File: gc3.kicad_pcb (KiCad board)
At the start: 4 copper layers, 99.2 x 77.2 mm, 202 parts, among them J1 JACK, J2 DM3AT-SF-PEJM5, P1 TESTPOINT, P10 UART1, P11 GND, P12 GND, P13 GND, P14 GND, P15 TESTPOINT, P16 TEESTPOINT, P17 GPIO, P18 USB_A, P19 USB_OTG, P2 TESTPOINT, P3 TESTPOINT, P4 TESTPOINT, P5 TESTPOINT, P6 TESTPOINT, P7 LCD, P8 JTAG, P9 UART0, SW1 PWR_ON, SW2 RESET, SW3 VOL+, SW4 VOL-, SW5 MENU, SW6 ENTER, SW7 HOME, U1 TPS62290, U2 axp209, U3 TPS62290, U4 a13, U5 h5tq2g63bfr, U6 TPS2552, U8 TPS2552, Y1 24MHz/20pF/20ppm

Commit message: Fix : bug fix
Parts:
- added ?: , via:via, F.Cu at (132.8, 58.9)
- added ?: , via:via, F.Cu at (114.8, 70.7)
- added ?: , via:via, F.Cu at (189.6, 114.9)
- added ?: , via:via, F.Cu at (195.4, 109.5)
- added ?: , via:via, F.Cu at (195.8, 113.4)
- added ?: , via:via, F.Cu at (195.8, 116.8)
- added ?: , via:via, F.Cu at (195.7, 120.8)
- added ?: , via:via, F.Cu at (195.8, 124.2)
- added ?: , via:via, F.Cu at (195.8, 128.0)
- added ?: , via:via, F.Cu at (195.8, 130.7)
- added ?: , via:via, F.Cu at (194.8, 111.6)
- added ?: , via:via, F.Cu at (194.8, 115.1)
- added ?: , via:via, F.Cu at (124.5, 67.5)
- added ?: , via:via, F.Cu at (194.8, 118.8)
- added ?: , via:via, F.Cu at (194.8, 122.7)
- added ?: , via:via, F.Cu at (194.8, 126.5)
- added ?: , via:via, F.Cu at (194.5, 130.7)
- added ?: , via:via, F.Cu at (197.8, 134.3)
- added ?: , via:via, F.Cu at (115.9, 104.3)
- added ?: , via:via, F.Cu at (118.5, 103.8)
- added ?: , via:via, F.Cu at (121.4, 103.8)
- added ?: , via:via, F.Cu at (125.2, 103.9)
- added ?: , via:via, F.Cu at (130.5, 103.8)
- added ?: , via:via, F.Cu at (131.7, 64.2)
- added ?: , via:via, F.Cu at (143.0, 103.8)
- added ?: , via:via, F.Cu at (118.6, 106.9)
- added ?: , via:via, F.Cu at (123.5, 107.1)
- added ?: , via:via, F.Cu at (128.7, 107.1)
- added ?: , via:via, F.Cu at (133.3, 107.1)
- added ?: , via:via, F.Cu at (137.3, 107.1)
- added ?: , via:via, F.Cu at (142.0, 107.1)
- added ?: , via:via, F.Cu at (111.3, 106.5)
- added ?: , via:via, F.Cu at (144.4, 107.5)
- added ?: , via:via, F.Cu at (144.4, 110.9)
- added ?: , via:via, F.Cu at (136.9, 64.2)
- added ?: , via:via, F.Cu at (144.4, 114.7)
- added ?: , via:via, F.Cu at (139.6, 111.2)
- added ?: , via:via, F.Cu at (132.5, 112.2)
- added ?: , via:via, F.Cu at (125.4, 112.0)
- added ?: , via:via, F.Cu at (119.1, 112.1)
- added ?: , via:via, F.Cu at (130.1, 117.2)
- added ?: , via:via, F.Cu at (122.7, 117.5)
- added ?: , via:via, F.Cu at (118.0, 116.9)
- added ?: , via:via, F.Cu at (109.1, 107.7)
- added ?: , via:via, F.Cu at (109.1, 112.9)
- added ?: , via:via, F.Cu at (131.1, 69.2)
- added ?: , via:via, F.Cu at (109.1, 117.3)
- added ?: , via:via, F.Cu at (109.1, 124.5)
- added ?: , via:via, F.Cu at (109.1, 130.8)
- added ?: , via:via, F.Cu at (109.1, 134.3)
- added ?: , via:via, F.Cu at (116.6, 134.3)
- added ?: , via:via, F.Cu at (120.5, 134.3)
- added ?: , via:via, F.Cu at (128.4, 132.9)
- added ?: , via:via, F.Cu at (137.2, 133.1)
- added ?: , via:via, F.Cu at (133.2, 133.0)
- added ?: , via:via, F.Cu at (132.9, 122.2)
- added ?: , via:via, F.Cu at (142.0, 69.7)
- added ?: , via:via, F.Cu at (138.2, 125.8)
- added ?: , via:via, F.Cu at (137.4, 129.8)
- added ?: , via:via, F.Cu at (133.9, 127.1)
- added ?: , via:via, F.Cu at (127.0, 121.9)
- added ?: , via:via, F.Cu at (127.9, 128.2)
- added ?: , via:via, F.Cu at (122.7, 125.2)
- added ?: , via:via, F.Cu at (119.4, 124.8)
- added ?: , via:via, F.Cu at (117.0, 119.6)
- added ?: , via:via, F.Cu at (117.5, 124.8)
- added ?: , via:via, F.Cu at (119.1, 128.0)
- added ?: , via:via, F.Cu at (137.6, 75.6)
- added ?: , via:via, F.Cu at (115.5, 118.0)
- added ?: , via:via, F.Cu at (115.4, 114.7)
- added ?: , via:via, F.Cu at (140.6, 75.2)
- added ?: , via:via, F.Cu at (142.1, 79.4)
- added ?: , via:via, F.Cu at (145.5, 82.1)
- added ?: , via:via, F.Cu at (127.7, 58.9)
- added ?: , via:via, F.Cu at (143.9, 82.1)
- added ?: , via:via, F.Cu at (129.3, 73.7)
- added ?: , via:via, F.Cu at (146.1, 71.9)
- added ?: , via:via, F.Cu at (109.2, 73.5)
- added ?: , via:via, F.Cu at (109.3, 78.3)
- added ?: , via:via, F.Cu at (109.2, 86.3)
- added ?: , via:via, F.Cu at (126.4, 79.6)
- added ?: , via:via, F.Cu at (116.8, 81.3)
- added ?: , via:via, F.Cu at (123.5, 82.4)
- added ?: , via:via, F.Cu at (123.5, 84.0)
- added ?: , via:via, F.Cu at (120.7, 59.0)
- added ?: , via:via, F.Cu at (127.1, 86.2)
- added ?: , via:via, F.Cu at (120.9, 84.7)
- added ?: , via:via, F.Cu at (145.5, 79.1)
- added ?: , via:via, F.Cu at (134.7, 84.0)
- added ?: , via:via, F.Cu at (130.1, 76.8)
- added ?: , via:via, F.Cu at (150.0, 69.5)
- added ?: , via:via, F.Cu at (112.0, 93.0)
- added ?: , via:via, F.Cu at (120.8, 91.0)
- added ?: , via:via, F.Cu at (116.0, 97.3)
- added ?: , via:via, F.Cu at (137.2, 84.2)
- added ?: , via:via, F.Cu at (115.0, 59.0)
- added ?: , via:via, F.Cu at (136.2, 90.4)
- added ?: , via:via, F.Cu at (144.9, 86.7)
- added ?: , via:via, F.Cu at (144.4, 92.1)
- added ?: , via:via, F.Cu at (143.8, 89.8)
- added ?: , via:via, F.Cu at (146.5, 89.8)
- added ?: , via:via, F.Cu at (143.9, 94.4)
- added ?: , via:via, F.Cu at (140.9, 94.6)
- added ?: , via:via, F.Cu at (143.9, 97.4)
- added ?: , via:via, F.Cu at (139.4, 98.2)
- added ?: , via:via, F.Cu at (135.4, 101.5)
- added ?: , via:via, F.Cu at (109.3, 59.0)
- added ?: , via:via, F.Cu at (140.0, 101.5)
- added ?: , via:via, F.Cu at (137.8, 101.5)
- added ?: , via:via, F.Cu at (182.6, 58.9)
- added ?: , via:via, F.Cu at (186.8, 58.9)
- added ?: , via:via, F.Cu at (189.9, 58.8)
- added ?: , via:via, F.Cu at (193.9, 61.9)
- added ?: , via:via, F.Cu at (196.6, 58.9)
- added ?: , via:via, F.Cu at (199.6, 61.6)
- added ?: , via:via, F.Cu at (202.7, 58.9)
- added ?: , via:via, F.Cu at (206.6, 58.8)
- added ?: , via:via, F.Cu at (109.3, 66.5)
- added ?: , via:via, F.Cu at (185.6, 64.8)
- added ?: , via:via, F.Cu at (180.6, 66.9)
- added ?: , via:via, F.Cu at (160.6, 73.5)
- added ?: , via:via, F.Cu at (163.1, 71.0)
- added ?: , via:via, F.Cu at (162.9, 73.6)
- added ?: , via:via, F.Cu at (196.2, 70.1)
- added ?: , via:via, F.Cu at (193.9, 72.3)
- added ?: , via:via, F.Cu at (188.4, 68.4)
- added ?: , via:via, F.Cu at (206.6, 73.4)
- added ?: , via:via, F.Cu at (206.6, 77.8)
- added ?: , via:via, F.Cu at (109.2, 62.9)
- added ?: , via:via, F.Cu at (206.6, 83.9)
- added ?: , via:via, F.Cu at (201.2, 70.8)
- added ?: , via:via, F.Cu at (202.8, 76.4)
- added ?: , via:via, F.Cu at (197.9, 76.6)
- added ?: , via:via, F.Cu at (193.0, 77.7)
- added ?: , via:via, F.Cu at (190.5, 84.9)
- added ?: , via:via, F.Cu at (192.8, 88.4)
- added ?: , via:via, F.Cu at (206.4, 88.4)
- added ?: , via:via, F.Cu at (197.4, 88.1)
- added ?: , via:via, F.Cu at (201.4, 89.2)
- added ?: , via:via, F.Cu at (153.9, 58.9)
- added ?: , via:via, F.Cu at (199.0, 92.7)
- added ?: , via:via, F.Cu at (206.5, 96.1)
- added ?: , via:via, F.Cu at (203.5, 97.4)
- added ?: , via:via, F.Cu at (200.0, 96.4)
- added ?: , via:via, F.Cu at (206.6, 104.4)
- added ?: , via:via, F.Cu at (202.6, 104.4)
- added ?: , via:via, F.Cu at (198.3, 105.5)
- added ?: , via:via, F.Cu at (206.6, 111.7)
- added ?: , via:via, F.Cu at (206.6, 119.1)
- added ?: , via:via, F.Cu at (203.0, 111.7)
- added ?: , via:via, F.Cu at (149.2, 59.0)
- added ?: , via:via, F.Cu at (198.6, 111.7)
- added ?: , via:via, F.Cu at (203.3, 119.0)
- added ?: , via:via, F.Cu at (198.5, 119.0)
- added ?: , via:via, F.Cu at (206.5, 127.6)
- added ?: , via:via, F.Cu at (203.6, 126.2)
- added ?: , via:via, F.Cu at (198.4, 127.7)
- added ?: , via:via, F.Cu at (206.6, 134.3)
- added ?: , via:via, F.Cu at (202.0, 134.3)
- added ?: , via:via, F.Cu at (198.6, 132.8)
- added ?: , via:via, F.Cu at (193.5, 134.3)
- C1: value 120uF/16V -> 100uF
- C78, C97: value 120uF -> 100uF
Routing:
- net GND: track 1225.8 -> 299.7 mm, vias 327 -> 139
- net (no net): track 15.4 -> 0.31 mm, vias 11 -> 0
Other:
- board text added: "RX"
- board text added: "TX"

Commit message: Temp : Temp commit for before Update4
Parts:
- C10, C11, C12, C13, C14, C15, C16, C17, C18, C19, C2, C20, C21, C22, C23, C24, C25, C26, C28, C29, C3, C30, C31, C32, C33, C34, C35, C36, C38, C39, C4, C40, C41, C42, C43, C44, C45, C46, C47, C48, C49, C5, C50, C51, C52, C53, C54, C55, C56, C57, C58, C59, C6, C60, C61, C62, C63, C64, C65, C66, C67, C68, C69, C7, C70, C71, C72, C73, C74, C75, C76, C79, C8, C80, C81, C82, C83, C84, C85, C86, C87, C88, C89, C9, C90, C91, C92, C93, C95, C96: footprint Capacitors_SMD:C_0603 -> COMMON0603:Common_0603
- JP1, R1, R10, R11, R12, R13, R15, R16, R17, R18, R19, R2, R20, R21, R22, R23, R24, R25, R26, R27, R28, R29, R3, R30, R31, R32, R33, R34, R35, R36, R37, R38, R39, R4, R40, R41, R42, R5, R56, R6, R66, R68, R69, R7, R70, R71, R72, R73, R74, R8, R9: footprint Resistors_SMD:R_0603 -> COMMON0603:Common_0603
- moved J2 7.80 mm to (198.8, 75.7)
- moved RA1 1.01 mm to (171.4, 100.8)
- moved RA10 1.01 mm to (188.2, 93.3)
- moved RA7 1.01 mm to (194.0, 96.5)
- moved RA3 1.00 mm to (175.4, 103.5)
- moved RA8 1.00 mm to (186.7, 96.6)
- moved RA5 0.99 mm to (192.1, 93.2)
- moved RA6 0.99 mm to (190.2, 96.5)
- moved RA4 0.99 mm to (162.4, 116.3)
- moved RA9 0.98 mm to (184.4, 99.4)
- moved RA2 0.98 mm to (162.4, 119.1)
- moved C34 0.12 mm to (151.2, 87.8)
Routing:
- net /mpu_ddr3/PIN39/USBH_EN: track 143.1 -> 144.3 mm

Commit message: Temp : temo commit for finish DDR3 routing
Parts:
- removed ? (x161): , via:via
- removed R30, R31, R32, R33, R34: 24R, COMMON0603:Common_0603
- added R14: 22R, Resistors_SMD:R_0201, F.Cu at (168.9, 100.9)
- added RA11: 22R, EXB28V:EXB18V, F.Cu at (170.3, 100.0)
- C58, C61, R26: moved to B.Cu
- C70, C72, C73, C74, C82, C89, C91, C92, C93: footprint COMMON0603:Common_0603 -> Capacitors_SMD:C_0402
- C71, C83, C84, C85, C86, C87, C88, C90: footprint COMMON0603:Common_0603 -> Capacitors_SMD:C_0402; moved to B.Cu
- JP1: footprint COMMON0603:Common_0603 -> Resistors_SMD:R_0603
- R27, R28: footprint COMMON0603:Common_0603 -> Resistors_SMD:R_0201
- R29: value 24R -> 22R; footprint COMMON0603:Common_0603 -> Resistors_SMD:R_0201
- RA1, RA10, RA2, RA3, RA4, RA5, RA6, RA7, RA8, RA9: footprint EXB28V:EXB28V -> EXB28V:EXB18V
- U5: footprint MT41J256M16:BGA-96_pitch0.8mm_dia0.4mm -> FBGA96:FBGA96(HYNIX_SAMSUNG_512MX16_DDR3)
- moved R69 34.0 mm to (207.8, 152.9)
- moved C31 34.0 mm to (204.3, 152.9)
- moved C69 34.0 mm to (206.2, 152.8)
- moved C72 29.7 mm to (180.7, 152.3)
- moved C89 29.7 mm to (185.6, 152.0)
- moved C73 29.1 mm to (175.4, 151.6)
- moved C92 27.3 mm to (194.7, 146.9), turned to 0 degrees
- moved R68 27.1 mm to (206.2, 148.0)
- moved C68 27.1 mm to (204.4, 148.0)
- moved C70 26.2 mm to (186.0, 145.1)
- moved C93 25.1 mm to (197.9, 143.3), turned to 0 degrees
- moved C83 22.5 mm to (179.3, 103.6), turned to 0 degrees
- moved C90 22.0 mm to (176.4, 103.6), turned to 0 degrees
- moved C91 21.1 mm to (196.3, 138.8), turned to 0 degrees
- moved C84 20.3 mm to (168.7, 103.5), turned to 180 degrees
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Connections:
- net /mpu_ddr3/+5V_USB_OTG renamed /+5V_USB_OTG
- net /mpu_ddr3/CK renamed /mpu_ddr3/CK_P
- net /mpu_ddr3/CKN renamed /mpu_ddr3/CK_N
- net /mpu_ddr3/NMI_N renamed /NMI_N
- net /mpu_ddr3/RESET_N renamed /RESET_N
- net /mpu_ddr3/SCK renamed /mpu_ddr3/SCK_P
- net /mpu_ddr3/SCKN renamed /mpu_ddr3/SCK_N
- U4 pad 31: /mpu_ddr3/SDQS0 -> /mpu_ddr3/SDQS0_P
- U4 pad 32: /mpu_ddr3/SDQS0N -> /mpu_ddr3/SDQS0_N
- U4 pad 33: /mpu_ddr3/SDQS1 -> /mpu_ddr3/SDQS1_P
- U4 pad 34: /mpu_ddr3/SDQS1N -> /mpu_ddr3/SDQS1_N
- U5 pad B7: /mpu_ddr3/DQS1N -> /mpu_ddr3/DQS1_N
- U5 pad C7: /mpu_ddr3/DQS1 -> /mpu_ddr3/DQS1_P
- U5 pad F3: /mpu_ddr3/DQS0 -> /mpu_ddr3/DQS0_P
- U5 pad G3: /mpu_ddr3/DQS0N -> /mpu_ddr3/DQS0_N
Routing:
- net +1.5V: track 240.3 -> 9.25 mm, vias 43 -> 2
- net +3.0VA: track 166.9 -> 6.87 mm, vias 4 -> 1
- net +5V: track 179.9 -> 38.4 mm
- net /mpu_ddr3/PIN7: track 184.4 -> 66.2 mm, vias 2 -> 1
- net GND: track 299.9 -> 200.1 mm, vias 139 -> 80
- net /mpu_ddr3/PIN36: track 84.3 -> 0.00 mm, vias 2 -> 0
- net /mpu_ddr3/PIN11/TWI1-SDA: track 83.7 -> 0.00 mm, vias 1 -> 0
- net /mpu_ddr3/PIN10/TWI1-SCK: track 81.4 -> 0.00 mm, vias 1 -> 0
- net /mpu_ddr3/PIN35: track 80.5 -> 0.00 mm, vias 2 -> 0
- net /mpu_ddr3/PIN34: track 77.8 -> 0.00 mm, vias 2 -> 0
- net /mpu_ddr3/PIN8: track 101.3 -> 24.6 mm, vias 1 -> 0
- net /mpu_ddr3/PIN33: track 75.6 -> 0.00 mm, vias 2 -> 0
- net PIN4/TWI0-SCK: track 140.9 -> 67.7 mm, vias 3 -> 2
- net /mpu_ddr3/PIN32: track 73.0 -> 0.00 mm, vias 2 -> 0
- net /mpu_ddr3/PIN6/PWM0: track 98.8 -> 26.5 mm, vias 1 -> 0
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Other:
- board size 99.2 x 77.2 mm -> 99.1 x 77.1 mm
- copper layers 4 -> 6
- rule trace_min: 0.127 -> 0.1

Commit message: Temp : temp commit, finish routing for Update4
Parts:
- removed R70: 8.2k/1%, COMMON0603:Common_0603
- removed R71: 10k/1%, COMMON0603:Common_0603
- removed R72: 11k/1%, COMMON0603:Common_0603
- removed R73: 13k/1%, COMMON0603:Common_0603
- removed SW4: VOL-, Buttons_Switches_SMD:SW_SPST_FSMSM
- removed SW5: MENU, Buttons_Switches_SMD:SW_SPST_FSMSM
- removed SW6: ENTER, Buttons_Switches_SMD:SW_SPST_FSMSM
- removed SW7: HOME, Buttons_Switches_SMD:SW_SPST_FSMSM
- C31, C52, C58, C61, C62, C68, C69: footprint COMMON0603:Common_0603 -> Capacitors_SMD:C_0402
- C51: footprint COMMON0603:Common_0603 -> Capacitors_SMD:C_0402; moved to B.Cu
- C70, C72, C73, C89, C91, C92, C93: moved to B.Cu
- R16: value 100k -> 100k/1%
- R26: moved to F.Cu
- R68, R69: footprint COMMON0603:Common_0603 -> Resistors_SMD:R_0402
- SW3: value VOL+ -> UBOOT
- moved C89 50.8 mm to (174.0, 102.5), turned to 90 degrees
- moved R69 49.8 mm to (175.6, 115.0)
- moved C69 49.4 mm to (174.2, 115.0)
- moved C31 49.2 mm to (172.9, 115.0)
- moved C73 46.2 mm to (165.8, 106.4), turned to 180 degrees
- moved C92 46.1 mm to (169.9, 108.1), turned to 180 degrees
- moved C91 45.8 mm to (165.8, 104.7), turned to 180 degrees
- moved C72 45.2 mm to (166.0, 109.5), turned to 180 degrees
- moved R68 43.3 mm to (178.2, 115.0)
- moved C93 43.2 mm to (182.2, 103.0)
- moved C68 42.9 mm to (176.9, 115.0)
- moved R16 41.4 mm to (189.3, 91.9), turned to 90 degrees
- moved C79 40.2 mm to (190.9, 91.9), turned to 90 degrees
- moved R56 35.5 mm to (192.5, 91.9)
- moved C70 34.1 mm to (174.1, 113.1)
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Connections:
- R56 pad 1: Net-(R56-Pad1) -> /mpu_ddr3/UBOOT
- SW3 pad 2: Net-(R56-Pad1) -> /mpu_ddr3/UBOOT
Routing:
- net /mpu_ddr3/UBOOT: track 0.00 -> 67.1 mm, vias 0 -> 2
- net +3.0VA: track 6.87 -> 72.0 mm, vias 1 -> 3
- net /mpu_ddr3/PIN36: track 0.00 -> 64.2 mm, vias 0 -> 2
- net /mpu_ddr3/PIN7: track 66.2 -> 130.2 mm, vias 1 -> 3
- net /mpu_ddr3/PIN35: track 0.00 -> 62.2 mm, vias 0 -> 1
- net /mpu_ddr3/PIN34: track 0.00 -> 56.9 mm, vias 0 -> 1
- net /mpu_ddr3/PIN29: track 0.00 -> 56.6 mm, vias 0 -> 1
- net /mpu_ddr3/PIN33: track 0.00 -> 56.5 mm, vias 0 -> 2
- net /mpu_ddr3/PIN8: track 24.6 -> 80.2 mm, vias 0 -> 1
- net /mpu_ddr3/PIN30: track 0.00 -> 55.0 mm, vias 0 -> 1
- net /mpu_ddr3/PIN6/PWM0: track 26.5 -> 81.4 mm, vias 0 -> 1
- net PIN5/TWI0-SDA: track 69.3 -> 124.1 mm, vias 2 -> 3
- net PIN4/TWI0-SCK: track 67.7 -> 122.0 mm, vias 2 -> 3
- net /mpu_ddr3/PIN32: track 0.00 -> 50.5 mm, vias 0 -> 2
- net /mpu_ddr3/PIN31: track 0.06 -> 49.2 mm, vias 0 -> 2
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Other:
- board size 99.1 x 77.1 mm -> 99.1 x 66.8 mm
- board text added: "UBOOT"
- board text removed: "ENTER"
- board text removed: "HOME"
- board text removed: "MENU"
- board text removed: "VOL+"
- board text removed: "VOL-"
