File: mpu_ddr3.sch (KiCad schematic (older format))
At the start: 136 parts, among them J2 DM3AT-SF-PEJM5, P10 UART1, P17 GPIO, P18 USB_A, P19 USB_OTG, P7 LCD, P8 JTAG, P9 UART0, SW3 VOL+, SW4 VOL-, SW5 MENU, SW6 ENTER, SW7 HOME, U4 a13, U5 h5tq2g63bfr, U6 TPS2552, U8 TPS2552, Y1 24MHz/20pF/10ppm

Commit message: clean sch and add resistor array
Parts:
- removed C28, C31, C80, C81, C83, C84, C85, C86, C88, C89, C90, C91, C92, C93: 0.1uF, symbol C-RESCUE-gc3
- removed C29, C30, C32, C33, C35, C38, C40, C42, C44, C45, C46, C47, C49, C52, C61: 0.1uF/6.3V, SMD_Packages:SMD-0603_c, symbol C-RESCUE-gc3
- removed C34, C43, C51, C65: 22uF/6.3V, SMD_Packages:SMD-0603_c, symbol C-RESCUE-gc3
- removed C36, C39, C41, C48, C50, C53, C55, C58, C62: 10uF/6.3V, SMD_Packages:SMD-0603_c, symbol C-RESCUE-gc3
- removed C54: 1uF/6.3V, SMD_Packages:SMD-0603_c, symbol C-RESCUE-gc3
- removed C56, C57, C63, C64: 1nF, SMD_Packages:SMD-0603_c, symbol C-RESCUE-gc3
- removed C66, C68, C69, C70, C71, C72, C73, C74: 0.1uF, SMD_Packages:SMD-0603_c, symbol C-RESCUE-gc3
- removed C79: 1nF, symbol C-RESCUE-gc3
- removed C82, C87: 22uF/6.3V, symbol C-RESCUE-gc3
- removed R14: JUMPER, symbol R-RESCUE-gc3
- removed R16: 100k, symbol R-RESCUE-gc3
- removed R17: 200k/1%, symbol R-RESCUE-gc3
- removed R18, R20, R21, R22, R23, R24, R25: 47k, symbol R-RESCUE-gc3
- removed R19, R68, R69, R74: 2k/1%, symbol R-RESCUE-gc3
- removed R26, R66: 240R/1%, symbol R-RESCUE-gc3
- removed R27, R28, R29, R30, R31, R32, R33, R34: 24R, symbol R-RESCUE-gc3
- removed R56: 6.8k/1%, symbol R-RESCUE-gc3
- removed R70: 8.2k/1%, symbol R-RESCUE-gc3
- removed R71: 10k/1%, symbol R-RESCUE-gc3
- removed R72: 11k/1%, symbol R-RESCUE-gc3
- removed R73: 13k/1%, symbol R-RESCUE-gc3
- removed RP1, RP10, RP2, RP3, RP4, RP5, RP6, RP7, RP8, RP9: R_PACK4, symbol R_PACK4
- added C28, C31, C47, C66, C68, C69, C70, C71, C72, C73, C74, C80, C81, C83, C84, C85, C86, C88, C89, C90, C91, C92, C93: 0.1uF, Capacitors_SMD:C_0603, symbol C
- added C29, C30, C32, C33, C35, C38, C40, C42, C44, C45, C46, C49, C52, C53, C54, C61: 0.1uF/6.3V, Capacitors_SMD:C_0603, symbol C
- added C34, C43, C51, C65, C82, C87: 22uF/6.3V, Capacitors_SMD:C_0603, symbol C
- added C36, C39, C41, C48, C50, C55, C58, C62: 10uF/6.3V, Capacitors_SMD:C_0603, symbol C
- added C56, C57, C63, C64, C79: 1uF, Capacitors_SMD:C_0603, symbol C
- added R14: JUMPER, Resistors_SMD:R_0603, symbol R
- added R16: 100k, Resistors_SMD:R_0603, symbol R
- added R17: 200k/1%, Resistors_SMD:R_0603, symbol R
- added R18, R20, R21, R22, R23, R24, R25: 47k, Resistors_SMD:R_0603, symbol R
- added R19, R68, R69, R74: 2k/1%, Resistors_SMD:R_0603, symbol R
- added R26, R66: 240R/1%, Resistors_SMD:R_0603, symbol R
- added R27, R28, R29, R30, R31, R32, R33, R34: 24R, Resistors_SMD:R_0603, symbol R
- added R56: 6.8k/1%, Resistors_SMD:R_0603, symbol R
- added R70: 8.2k/1%, Resistors_SMD:R_0603, symbol R
- added R71: 10k/1%, Resistors_SMD:R_0603, symbol R
- added R72: 11k/1%, Resistors_SMD:R_0603, symbol R
- added R73: 13k/1%, Resistors_SMD:R_0603, symbol R
- added RA1, RA10, RA2, RA3, RA4, RA5, RA6, RA7, RA8, RA9: 22R, EXB28V:EXB28V, symbol RA
- C59, C60, C67, C75, C76, C78, C95, C96: footprint (none) -> Capacitors_SMD:C_0603
- C97: footprint (none) -> Capacitors_ThroughHole:C_Radial_D5_L11_P2
- J2: footprint (none) -> DM3AT-SF-PEJM5:DM3AT-SF-PEJM5
- L5, L7, L8, L9: footprint (none) -> Resistors_SMD:R_0805
- P17: footprint (none) -> Pin_Headers:Pin_Header_Straight_2x20
- P18: footprint (none) -> Connect:USB_A_Vertical
- P19: footprint (none) -> Connect:USB_Micro-B
- P7: footprint Pin_Headers:Pin_Header_Angled_2x20 -> Pin_Headers:Pin_Header_Straight_2x20
- R35, R36, R37, R38, R39, R40, R41, R42: footprint (none) -> Resistors_SMD:R_0603
- SW3, SW4, SW5, SW6, SW7: footprint (none) -> Buttons_Switches_SMD:SW_SPST_FSMSM
- U4: footprint (none) -> A13:LQFP-176_20x20mm_Pitch0.4mm
- U5: footprint (none) -> MT41J256M16:BGA-96_pitch0.8mm_dia0.4mm
- U6, U8: footprint (none) -> Housings_SOT-23_SOT-143_TSOT-6:SOT-23-6
- Y1: value 24MHz/20pF/10ppm -> 24MHz/20pF/20ppm; footprint (none) -> ECX32:ecx32
Connections:
- net labels removed: +3.3V-RESCUE-gc3
- wire segments 731 -> 684
Other:
- note added: "LCD\n"
- note removed: "LCD"

Commit message: commit before cleanup all footprint
Changed lines of the file:
@@
 LIBS:valves
 LIBS:a13
-LIBS:mp1482ds
 LIBS:3.0VA
 LIBS:1.2V_CPU
 LIBS:1.2V_INT
 LIBS:+1.5V
-LIBS:pcf8563t5
 LIBS:usd
 LIBS:axp209
@@
 LIBS:crystall
 LIBS:resistorarray
+LIBS:blueninja
 LIBS:gc3-cache
 EELAYER 25 0
@@
 Text Label 6590 12695 2    60   ~ 0
 SVREF
-Text Notes 8195 840  0    60   ~ 0
+Text Notes 7935 1025 0    60   ~ 0
 2GB 128M 8Bank x16
 Text Label 9750 3305 0    60   ~ 0
@@
 P 3570 4800
 F 0 "#PWR064" H 3570 4550 50  0001 C CNN
-F 1 "GND" V 3540 4630 50  0000 C CNN
+F 1 "GND" V 3570 4615 50  0000 C CNN
 F 2 "" H 3570 4800 60  0000 C CNN
 F 3 "" H 3570 4800 60  0000 C CNN
@@
 P 3180 4800
 F 0 "#PWR065" H 3180 4550 50  0001 C CNN
-F 1 "GND" V 3240 4645 50  0000 C CNN
+F 1 "GND" V 3180 4615 50  0000 C CNN
 F 2 "" H 3180 4800 60  0000 C CNN
 F 3 "" H 3180 4800 60  0000 C CNN
@@
 P 1815 5405
 F 0 "#PWR067" H 1815 5155 50  0001 C CNN
-F 1 "GND" V 1880 5240 50  0000 C CNN
+F 1 "GND" V 1815 5215 50  0000 C CNN
 F 2 "" H 1815 5405 60  0000 C CNN
 F 3 "" H 1815 5405 60  0000 C CNN
@@
 P 1885 5810
 F 0 "#PWR071" H 1885 5560 50  0001 C CNN
-F 1 "GND" H 1885 5660 50  0000 C CNN
+F 1 "GND" V 1885 5625 50  0000 C CNN
 F 2 "" H 1885 5810 60  0000 C CNN
 F 3 "" H 1885 5810 60  0000 C CNN
@@
 P 1815 4225
 F 0 "C62" V 1885 4320 50  0000 L CNN
-F 1 "10uF/6.3V" V 1970 4000 50  0000 L CNN
+F 1 "10uF/6.3V" V 1950 3910 50  0000 L CNN
 F 2 "Capacitors_SMD:C_0603" H 1853 4075 30  0001 C CNN
 F 3 "" H 1815 4225 60  0000 C CNN
@@
 P 10075 10820
 F 0 "#PWR091" H 10075 10570 50  0001 C CNN
-F 1 "GND" V 10105 10635 50  0000 C CNN
+F 1 "GND" V 10075 10630 50  0000 C CNN
 F 2 "" H 10075 10820 60  0000 C CNN
 F 3 "" H 10075 10820 60  0000 C CNN
@@
 P 8350 5355
 F 0 "#PWR097" H 8350 5105 50  0001 C CNN
-F 1 "GND" V 8380 5165 50  0000 C CNN
+F 1 "GND" V 8350 5165 50  0000 C CNN
 F 2 "" H 8350 5355 60  0000 C CNN
 F 3 "" H 8350 5355 60  0000 C CNN
@@
 $EndComp
 $Comp
-L +1.5V #PWR0105
+L +1.5V #PWR0104
 U 1 1 5668D19B
 P 10965 7670
-F 0 "#PWR0105" H 10965 7810 20  0001 C CNN
+F 0 "#PWR0104" H 10965 7810 20  0001 C CNN
 F 1 "+1.5V" H 10965 7780 30  0000 C CNN
 F 2 "" H 10965 7670 60  0000 C CNN
@@
 RESET
 $Comp
-L GND #PWR0106
+L GND #PWR0105
 U 1 1 568ADD15
 P 9680 6555
-F 0 "#PWR0106" H 9680 6305 50  0001 C CNN
+F 0 "#PWR0105" H 9680 6305 50  0001 C CNN
 F 1 "GND" V 9735 6395 50  0000 C CNN
 F 2 "" H 9680 6555 60  0000 C CNN
@@
 	7275 6010 7275 4685
 $Comp
-L GND #PWR0107
+L GND #PWR0106
 U 1 1 568C7349
 P 8890 8975
-F 0 "#PWR0107" H 8890 8725 50  0001 C CNN
+F 0 "#PWR0106" H 8890 8725 50  0001 C CNN
 F 1 "GND" V 8890 8790 50  0000 C CNN
 F 2 "" H 8890 8975 60  0000 C CNN
@@
 $EndComp
 $Comp
-L +5V #PWR0108
+L +5V #PWR0107
 U 1 1 568C9B7A
 P 8065 8975
-F 0 "#PWR0108" H 8065 8825 50  0001 C CNN
+F 0 "#PWR0107" H 8065 8825 50  0001 C CNN
 F 1 "+5V" V 8065 9165 50  0000 C CNN
 F 2 "" H 8065 8975 60  0000 C CNN
@@
 $EndComp
 $Comp
-L +3.3V #PWR0109
+L +3.3V #PWR0108
 U 1 1 568CAA99
 P 8065 9075
-F 0 "#PWR0109" H 8065 8925 50  0001 C CNN
+F 0 "#PWR0108" H 8065 8925 50  0001 C CNN
 F 1 "+3.3V" V 8065 9300 50  0000 C CNN
 F 2 "" H 8065 9075 60  0000 C CNN
@@
 $EndComp
 $Comp
-L GND #PWR0110
+L GND #PWR0109
 U 1 1 569B3524
 P 2260 9990
-F 0 "#PWR0110" H 2260 9740 50  0001 C CNN
-F 1 "GND" V 2310 9830 50  0000 C CNN
+F 0 "#PWR0109" H 2260 9740 50  0001 C CNN
+F 1 "GND" V 2265 9790 50  0000 C CNN
 F 2 "" H 2260 9990 60  0000 C CNN
 F 3 "" H 2260 9990 60  0000 C CNN
@@
 $EndComp
 $Comp
-L GND #PWR0111
+L GND #PWR0110
 U 1 1 569E74F6
 P 8080 8215
-F 0 "#PWR0111" H 8080 7965 50  0001 C CNN
+F 0 "#PWR0110" H 8080 7965 50  0001 C CNN
 F 1 "GND" H 8080 8065 50  0000 C CNN
 F 2 "" H 8080 8215 60  0000 C CNN
@@
 $EndComp
 $Comp
-L +1.5V #PWR0112
+L +1.5V #PWR0111
 U 1 1 569E7F1E
 P 8080 7610
-F 0 "#PWR0112" H 8080 7750 20  0001 C CNN
+F 0 "#PWR0111" H 8080 7750 20  0001 C CNN
 F 1 "+1.5V" H 8080 7720 30  0000 C CNN
 F 2 "" H 8080 7610 60  0000 C CNN
@@
 $EndComp
 $Comp
-L GND #PWR0113
+L GND #PWR0112
 U 1 1 569FF78C
 P 9120 8215
-F 0 "#PWR0113" H 9120 7965 50  0001 C CNN
+F 0 "#PWR0112" H 9120 7965 50  0001 C CNN
 F 1 "GND" H 9120 8065 50  0000 C CNN
 F 2 "" H 9120 8215 60  0000 C CNN
@@
 $EndComp
 $Comp
-L +1.5V #PWR0114
+L +1.5V #PWR0113
 U 1 1 569FF792
 P 9120 7610
-F 0 "#PWR0114" H 9120 7750 20  0001 C CNN
+F 0 "#PWR0113" H 9120 7750 20  0001 C CNN
 F 1 "+1.5V" H 9120 7720 30  0000 C CNN
 F 2 "" H 9120 7610 60  0000 C CNN
@@
 $EndComp
 $Comp
-L GND #PWR0115
+L GND #PWR0114
 U 1 1 56A0197B
 P 10550 8220
-F 0 "#PWR0115" H 10550 7970 50  0001 C CNN
+F 0 "#PWR0114" H 10550 7970 50  0001 C CNN
 F 1 "GND" H 10550 8070 50  0000 C CNN
 F 2 "" H 10550 8220 60  0000 C CNN
@@
 $EndComp
 $Comp
-L +1.5V #PWR0116
+L +1.5V #PWR0115
 U 1 1 56A01981
 P 10550 7605
-F 0 "#PWR0116" H 10550 7745 20  0001 C CNN
+F 0 "#PWR0115" H 10550 7745 20  0001 C CNN
 F 1 "+1.5V" H 10550 7715 30  0000 C CNN
 F 2 "" H 10550 7605 60  0000 C CNN
@@
 	1605 11890 1355 11890
 $Comp
-L +5V #PWR0117
+L +5V #PWR0116
 U 1 1 56A45A51
 P 1450 9990
-F 0 "#PWR0117" H 1450 9840 50  0001 C CNN
+F 0 "#PWR0116" H 1450 9840 50  0001 C CNN
 F 1 "+5V" V 1450 10185 50  0000 C CNN
 F 2 "" H 1450 9990 60  0000 C CNN
@@
 	1450 9990 1605 9990
 $Comp
-L +3.3V #PWR0118
+L +3.3V #PWR0117
 U 1 1 56A48B5D
 P 1450 10090
-F 0 "#PWR0118" H 1450 9940 50  0001 C CNN
+F 0 "#PWR0117" H 1450 9940 50  0001 C CNN
 F 1 "+3.3V" V 1450 10310 50  0000 C CNN
 F 2 "" H 1450 10090 60  0000 C CNN
@@
 Connection ~ 7510 13820
 $Comp
-L GND #PWR0119
+L GND #PWR0118
 U 1 1 56AC091E
 P 9415 14560
-F 0 "#PWR0119" H 9415 14310 50  0001 C CNN
+F 0 "#PWR0118" H 9415 14310 50  0001 C CNN
 F 1 "GND" H 9415 14410 50  0000 C CNN
 F 2 "" H 9415 14560 60  0000 C CNN
@@
 Connection ~ 7880 14515
 $Comp
-L +3.0VA #PWR0120
+L +3.0VA #PWR0119
 U 1 1 56AC9BBB
 P 7030 13820
-F 0 "#PWR0120" H 7030 13780 30  0001 C CNN
+F 0 "#PWR0119" H 7030 13780 30  0001 C CNN
 F 1 "+3.0VA" V 7025 13995 30  0000 C CNN
 F 2 "" H 7030 13820 60  0000 C CNN
@@
 	1825 3400 1825 3525
 $Comp
-L GND #PWR0121
+L GND #PWR0120
 U 1 1 562E1106
 P 1825 3525
-F 0 "#PWR0121" H 1825 3275 50  0001 C CNN
+F 0 "#PWR0120" H 1825 3275 50  0001 C CNN
 F 1 "GND" H 1825 3375 50  0000 C CNN
 F 2 "" H 1825 3525 60  0000 C CNN
@@
 Connection ~ 9180 11950
 $Comp
-L +1.5V #PWR?
+L +1.5V #PWR0121
 U 1 1 56311B76
 P 10965 8185
-F 0 "#PWR?" H 10965 8325 20  0001 C CNN
+F 0 "#PWR0121" H 10965 8325 20  0001 C CNN
 F 1 "+1.5V" H 10965 8295 30  0000 C CNN
 F 2 "" H 10965 8185 60  0000 C CNN

Commit message: clean: all footprint
Parts:
- removed R14: JUMPER, Resistors_SMD:R_0603, symbol R
- C78: footprint Capacitors_SMD:C_0603 -> Capacitors_ThroughHole:C_Radial_D5_L11_P2
Connections:
- wire segments 684 -> 682
Changed lines of the file:
@@
 F 0 "C78" H 3775 13745 50  0000 L CNN
 F 1 "120uF" V 3805 13355 50  0000 L CNN
-F 2 "Capacitors_SMD:C_0603" H 3788 13495 30  0001 C CNN
+F 2 "Capacitors_ThroughHole:C_Radial_D5_L11_P2" H 3788 13495 30  0001 C CNN
 F 3 "" H 3750 13645 60  0000 C CNN
 	1    3750 13645
@@
 Connection ~ 6950 12695
 Connection ~ 6745 12695
-$Comp
-L R R14
-U 1 1 5668CB44
-P 10965 7935
-F 0 "R14" V 11045 7935 50  0000 C CNN
-F 1 "JUMPER" V 10885 7935 50  0000 C CNN
-F 2 "Resistors_SMD:R_0603" V 10895 7935 30  0001 C CNN
-F 3 "" H 10965 7935 30  0000 C CNN
-	1    10965 7935
-	1    0    0    -1
-$EndComp
-$Comp
-L +1.5V #PWR0104
-U 1 1 5668D19B
-P 10965 7670
-F 0 "#PWR0104" H 10965 7810 20  0001 C CNN
-F 1 "+1.5V" H 10965 7780 30  0000 C CNN
-F 2 "" H 10965 7670 60  0000 C CNN
-F 3 "" H 10965 7670 60  0000 C CNN
-	1    10965 7670
-	1    0    0    -1
-$EndComp
-Wire Wire Line
-	10965 7670 10965 7785
-Wire Wire Line
-	10965 8085 10965 8185
 Wire Wire Line
 	6675 1160 7175 1160
@@
 	9180 11845 9180 11950
 Connection ~ 9180 11950
-$Comp
-L +1.5V #PWR0121
-U 1 1 56311B76
-P 10965 8185
-F 0 "#PWR0121" H 10965 8325 20  0001 C CNN
-F 1 "+1.5V" H 10965 8295 30  0000 C CNN
-F 2 "" H 10965 8185 60  0000 C CNN
-F 3 "" H 10965 8185 60  0000 C CNN
-	1    10965 8185
-	-1   0    0    1
-$EndComp
 $EndSCHEMATC

Commit message: Fix : bug fix
Parts:
- C78, C97: value 120uF -> 100uF
Changed lines of the file:
@@
 P 3750 13645
 F 0 "C78" H 3775 13745 50  0000 L CNN
-F 1 "120uF" V 3805 13355 50  0000 L CNN
+F 1 "100uF" V 3805 13355 50  0000 L CNN
 F 2 "Capacitors_ThroughHole:C_Radial_D5_L11_P2" H 3788 13495 30  0001 C CNN
 F 3 "" H 3750 13645 60  0000 C CNN
@@
 P 3804 15115
 F 0 "C97" H 3829 15215 50  0000 L CNN
-F 1 "120uF" V 3859 14825 50  0000 L CNN
+F 1 "100uF" V 3859 14825 50  0000 L CNN
 F 2 "Capacitors_ThroughHole:C_Radial_D5_L11_P2" H 3842 14965 30  0001 C CNN
 F 3 "" H 3804 15115 60  0000 C CNN
@@
 RESET
 $Comp
-L GND #PWR0105
+L GND #PWR0104
 U 1 1 568ADD15
 P 9680 6555
-F 0 "#PWR0105" H 9680 6305 50  0001 C CNN
+F 0 "#PWR0104" H 9680 6305 50  0001 C CNN
 F 1 "GND" V 9735 6395 50  0000 C CNN
 F 2 "" H 9680 6555 60  0000 C CNN
@@
 	7275 6010 7275 4685
 $Comp
-L GND #PWR0106
+L GND #PWR0105
 U 1 1 568C7349
 P 8890 8975
-F 0 "#PWR0106" H 8890 8725 50  0001 C CNN
+F 0 "#PWR0105" H 8890 8725 50  0001 C CNN
 F 1 "GND" V 8890 8790 50  0000 C CNN
 F 2 "" H 8890 8975 60  0000 C CNN
@@
 $EndComp
 $Comp
-L +5V #PWR0107
+L +5V #PWR0106
 U 1 1 568C9B7A
 P 8065 8975
-F 0 "#PWR0107" H 8065 8825 50  0001 C CNN
+F 0 "#PWR0106" H 8065 8825 50  0001 C CNN
 F 1 "+5V" V 8065 9165 50  0000 C CNN
 F 2 "" H 8065 8975 60  0000 C CNN
@@
 $EndComp
 $Comp
-L +3.3V #PWR0108
+L +3.3V #PWR0107
 U 1 1 568CAA99
 P 8065 9075
-F 0 "#PWR0108" H 8065 8925 50  0001 C CNN
+F 0 "#PWR0107" H 8065 8925 50  0001 C CNN
 F 1 "+3.3V" V 8065 9300 50  0000 C CNN
 F 2 "" H 8065 9075 60  0000 C CNN
@@
 $EndComp
 $Comp
-L GND #PWR0109
+L GND #PWR0108
 U 1 1 569B3524
 P 2260 9990
-F 0 "#PWR0109" H 2260 9740 50  0001 C CNN
+F 0 "#PWR0108" H 2260 9740 50  0001 C CNN
 F 1 "GND" V 2265 9790 50  0000 C CNN
 F 2 "" H 2260 9990 60  0000 C CNN
@@
 $EndComp
 $Comp
-L GND #PWR0110
+L GND #PWR0109
 U 1 1 569E74F6
 P 8080 8215
-F 0 "#PWR0110" H 8080 7965 50  0001 C CNN
+F 0 "#PWR0109" H 8080 7965 50  0001 C CNN
 F 1 "GND" H 8080 8065 50  0000 C CNN
 F 2 "" H 8080 8215 60  0000 C CNN
@@
 $EndComp
 $Comp
-L +1.5V #PWR0111
+L +1.5V #PWR0110
 U 1 1 569E7F1E
 P 8080 7610
-F 0 "#PWR0111" H 8080 7750 20  0001 C CNN
+F 0 "#PWR0110" H 8080 7750 20  0001 C CNN
 F 1 "+1.5V" H 8080 7720 30  0000 C CNN
 F 2 "" H 8080 7610 60  0000 C CNN
@@
 $EndComp
 $Comp
-L GND #PWR0112
+L GND #PWR0111
 U 1 1 569FF78C
 P 9120 8215
-F 0 "#PWR0112" H 9120 7965 50  0001 C CNN
+F 0 "#PWR0111" H 9120 7965 50  0001 C CNN
 F 1 "GND" H 9120 8065 50  0000 C CNN
 F 2 "" H 9120 8215 60  0000 C CNN
@@
 $EndComp
 $Comp
-L +1.5V #PWR0113
+L +1.5V #PWR0112
 U 1 1 569FF792
 P 9120 7610
-F 0 "#PWR0113" H 9120 7750 20  0001 C CNN
+F 0 "#PWR0112" H 9120 7750 20  0001 C CNN
 F 1 "+1.5V" H 9120 7720 30  0000 C CNN
 F 2 "" H 9120 7610 60  0000 C CNN
@@
 $EndComp
 $Comp
-L GND #PWR0114
+L GND #PWR0113
 U 1 1 56A0197B
 P 10550 8220
-F 0 "#PWR0114" H 10550 7970 50  0001 C CNN
+F 0 "#PWR0113" H 10550 7970 50  0001 C CNN
 F 1 "GND" H 10550 8070 50  0000 C CNN
 F 2 "" H 10550 8220 60  0000 C CNN
@@
 $EndComp
 $Comp
-L +1.5V #PWR0115
+L +1.5V #PWR0114
 U 1 1 56A01981
 P 10550 7605
-F 0 "#PWR0115" H 10550 7745 20  0001 C CNN
+F 0 "#PWR0114" H 10550 7745 20  0001 C CNN
 F 1 "+1.5V" H 10550 7715 30  0000 C CNN
 F 2 "" H 10550 7605 60  0000 C CNN
@@
 	1605 11890 1355 11890
 $Comp
-L +5V #PWR0116
+L +5V #PWR0115
 U 1 1 56A45A51
 P 1450 9990
-F 0 "#PWR0116" H 1450 9840 50  0001 C CNN
+F 0 "#PWR0115" H 1450 9840 50  0001 C CNN
 F 1 "+5V" V 1450 10185 50  0000 C CNN
 F 2 "" H 1450 9990 60  0000 C CNN
@@
 	1450 9990 1605 9990
 $Comp
-L +3.3V #PWR0117
+L +3.3V #PWR0116
 U 1 1 56A48B5D
 P 1450 10090
-F 0 "#PWR0117" H 1450 9940 50  0001 C CNN
+F 0 "#PWR0116" H 1450 9940 50  0001 C CNN
 F 1 "+3.3V" V 1450 10310 50  0000 C CNN
 F 2 "" H 1450 10090 60  0000 C CNN
@@
 Connection ~ 7510 13820
 $Comp
-L GND #PWR0118
+L GND #PWR0117
 U 1 1 56AC091E
 P 9415 14560
-F 0 "#PWR0118" H 9415 14310 50  0001 C CNN
+F 0 "#PWR0117" H 9415 14310 50  0001 C CNN
 F 1 "GND" H 9415 14410 50  0000 C CNN
 F 2 "" H 9415 14560 60  0000 C CNN
@@
 Connection ~ 7880 14515
 $Comp
-L +3.0VA #PWR0119
+L +3.0VA #PWR0118
 U 1 1 56AC9BBB
 P 7030 13820
-F 0 "#PWR0119" H 7030 13780 30  0001 C CNN
+F 0 "#PWR0118" H 7030 13780 30  0001 C CNN
 F 1 "+3.0VA" V 7025 13995 30  0000 C CNN
 F 2 "" H 7030 13820 60  0000 C CNN
@@
 	1825 3400 1825 3525
 $Comp
-L GND #PWR0120
+L GND #PWR0119
 U 1 1 562E1106
 P 1825 3525
-F 0 "#PWR0120" H 1825 3275 50  0001 C CNN
+F 0 "#PWR0119" H 1825 3275 50  0001 C CNN
 F 1 "GND" H 1825 3375 50  0000 C CNN
 F 2 "" H 1825 3525 60  0000 C CNN

Commit message: Temp : Temp commit for before Update4
Parts:
- C28, C29, C30, C31, C32, C33, C34, C35, C36, C38, C39, C40, C41, C42, C43, C44, C45, C46, C47, C48, C49, C50, C51, C52, C53, C54, C55, C56, C57, C58, C59, C60, C61, C62, C63, C64, C65, C66, C67, C68, C69, C70, C71, C72, C73, C74, C75, C76, C79, C80, C81, C82, C83, C84, C85, C86, C87, C88, C89, C90, C91, C92, C93, C95, C96: footprint Capacitors_SMD:C_0603 -> COMMON0603:Common_0603
- R16, R17, R18, R19, R20, R21, R22, R23, R24, R25, R26, R27, R28, R29, R30, R31, R32, R33, R34, R35, R36, R37, R38, R39, R40, R41, R42, R56, R66, R68, R69, R70, R71, R72, R73, R74: footprint Resistors_SMD:R_0603 -> COMMON0603:Common_0603

Commit message: Temp : temo commit for finish DDR3 routing
Parts:
- removed R30, R31, R32, R33, R34: 24R, COMMON0603:Common_0603, symbol R
- added R14: 22R, Resistors_SMD:R_0201, symbol R
- added RA11: 22R, EXB28V:EXB18V, symbol RA
- C70, C71, C72, C73, C74, C82, C83, C84, C85, C86, C87, C88, C89, C90, C91, C92, C93: footprint COMMON0603:Common_0603 -> Capacitors_SMD:C_0402
- R27, R28: footprint COMMON0603:Common_0603 -> Resistors_SMD:R_0201
- R29: value 24R -> 22R; footprint COMMON0603:Common_0603 -> Resistors_SMD:R_0201
- RA1, RA10, RA2, RA3, RA4, RA5, RA6, RA7, RA8, RA9: footprint EXB28V:EXB28V -> EXB28V:EXB18V
- U5: footprint MT41J256M16:BGA-96_pitch0.8mm_dia0.4mm -> FBGA96:FBGA96(HYNIX_SAMSUNG_512MX16_DDR3)
Connections:
- net labels added: CK_N, CK_P, DQS0_N, DQS0_P, DQS1_N, DQS1_P, SCK_N, SCK_P, SDQS0_N, SDQS0_P, SDQS1_N, SDQS1_P
- net labels removed: CK, CKN, DQS0, DQS0N, DQS1, DQS1N, SCK, SCKN, SDQS0, SDQS0N, SDQS1, SDQS1N

Commit message: Temp : temp commit, finish routing for Update4
Parts:
- removed R70: 8.2k/1%, COMMON0603:Common_0603, symbol R
- removed R71: 10k/1%, COMMON0603:Common_0603, symbol R
- removed R72: 11k/1%, COMMON0603:Common_0603, symbol R
- removed R73: 13k/1%, COMMON0603:Common_0603, symbol R
- removed SW4: VOL-, Buttons_Switches_SMD:SW_SPST_FSMSM, symbol SW_PUSH
- removed SW5: MENU, Buttons_Switches_SMD:SW_SPST_FSMSM, symbol SW_PUSH
- removed SW6: ENTER, Buttons_Switches_SMD:SW_SPST_FSMSM, symbol SW_PUSH
- removed SW7: HOME, Buttons_Switches_SMD:SW_SPST_FSMSM, symbol SW_PUSH
- C31, C51, C52, C58, C61, C62, C68, C69: footprint COMMON0603:Common_0603 -> Capacitors_SMD:C_0402
- R16: value 100k -> 100k/1%
- R68, R69: footprint COMMON0603:Common_0603 -> Resistors_SMD:R_0402
- SW3: value VOL+ -> UBOOT
Connections:
- wire segments 682 -> 670
