File: mpu_ddr3.sch (KiCad schematic (older format))
At the start: 124 parts, among them J2 DM3AT-SF-PEJM5, P10 UART1, P17 GPIO, P18 USB_A, P19 USB_OTG, P7 LCD, P8 JTAG, P9 UART0, SW3 UBOOT, U4 a13, U5 h5tq2g63bfr, U6 TPS2552, U8 TPS2552, Y1 24MHz/20pF/20ppm

Commit message: Add : finish Update$
Parts:
- C29, C30, C32, C33, C34, C35, C36, C38, C39, C40, C41, C42, C43, C44, C47, C48, C49, C50, C66, C80, C81: footprint COMMON0603:Common_0603 -> Capacitors_SMD:C_0402
- R19, R26, R66, R74: footprint COMMON0603:Common_0603 -> Resistors_SMD:R_0402
Changed lines of the file:
@@
 F 0 "C66" V 6620 6070 50  0000 L CNN
 F 1 "0.1uF" V 6620 6345 50  0000 L CNN
-F 2 "COMMON0603:Common_0603" H 6693 6110 30  0001 C CNN
+F 2 "Capacitors_SMD:C_0402" H 6693 6110 30  0001 C CNN
 F 3 "" H 6655 6260 60  0000 C CNN
 	1    6655 6260
@@
 F 0 "R66" V 6260 6165 50  0000 C CNN
 F 1 "240R/1%" V 6365 6645 50  0000 C CNN
-F 2 "COMMON0603:Common_0603" V 6230 6360 30  0001 C CNN
+F 2 "Resistors_SMD:R_0402" V 6230 6360 30  0001 C CNN
 F 3 "" H 6300 6360 30  0000 C CNN
 	1    6300 6360
@@
 F 0 "C47" V 2335 6635 50  0000 L CNN
 F 1 "0.1uF" V 2335 6280 50  0000 L CNN
-F 2 "COMMON0603:Common_0603" H 2308 6400 30  0001 C CNN
+F 2 "Capacitors_SMD:C_0402" H 2308 6400 30  0001 C CNN
 F 3 "" H 2270 6550 60  0000 C CNN
 	1    2270 6550
@@
 F 0 "C29" V 1080 1300 50  0000 L CNN
 F 1 "0.1uF/6.3V" V 990 980 50  0000 L CNN
-F 2 "COMMON0603:Common_0603" H 1153 1095 30  0001 C CNN
+F 2 "Capacitors_SMD:C_0402" H 1153 1095 30  0001 C CNN
 F 3 "" H 1115 1245 60  0000 C CNN
 	1    1115 1245
@@
 F 0 "C30" V 1265 1310 50  0000 L CNN
 F 1 "0.1uF/6.3V" V 1235 765 50  0000 L CNN
-F 2 "COMMON0603:Common_0603" H 1343 1095 30  0001 C CNN
+F 2 "Capacitors_SMD:C_0402" H 1343 1095 30  0001 C CNN
 F 3 "" H 1305 1245 60  0000 C CNN
 	1    1305 1245
@@
 F 0 "C32" V 1455 1310 50  0000 L CNN
 F 1 "0.1uF/6.3V" V 1430 765 50  0000 L CNN
-F 2 "COMMON0603:Common_0603" H 1533 1095 30  0001 C CNN
+F 2 "Capacitors_SMD:C_0402" H 1533 1095 30  0001 C CNN
 F 3 "" H 1495 1245 60  0000 C CNN
 	1    1495 1245
@@
 F 0 "C33" V 1645 1310 50  0000 L CNN
 F 1 "0.1uF/6.3V" V 1830 1025 50  0000 L CNN
-F 2 "COMMON0603:Common_0603" H 1723 1095 30  0001 C CNN
+F 2 "Capacitors_SMD:C_0402" H 1723 1095 30  0001 C CNN
 F 3 "" H 1685 1245 60  0000 C CNN
 	1    1685 1245
@@
 F 0 "C34" H 820 2300 50  0000 L CNN
 F 1 "22uF/6.3V" V 750 1750 50  0000 L CNN
-F 2 "COMMON0603:Common_0603" H 833 2050 30  0001 C CNN
+F 2 "Capacitors_SMD:C_0402" H 833 2050 30  0001 C CNN
 F 3 "" H 795 2200 60  0000 C CNN
 	1    795  2200
@@
 F 0 "C35" H 1010 2300 50  0000 L CNN
 F 1 "0.1uF/6.3V" V 935 1725 50  0000 L CNN
-F 2 "COMMON0603:Common_0603" H 1023 2050 30  0001 C CNN
+F 2 "Capacitors_SMD:C_0402" H 1023 2050 30  0001 C CNN
 F 3 "" H 985 2200 60  0000 C CNN
 	1    985  2200
@@
 F 0 "C36" H 1200 2300 50  0000 L CNN
 F 1 "10uF/6.3V" V 1120 1745 50  0000 L CNN
-F 2 "COMMON0603:Common_0603" H 1213 2050 30  0001 C CNN
+F 2 "Capacitors_SMD:C_0402" H 1213 2050 30  0001 C CNN
 F 3 "" H 1175 2200 60  0000 C CNN
 	1    1175 2200
@@
 F 0 "C38" H 1390 2300 50  0000 L CNN
 F 1 "0.1uF/6.3V" V 1315 1720 50  0000 L CNN
-F 2 "COMMON0603:Common_0603" H 1403 2050 30  0001 C CNN
+F 2 "Capacitors_SMD:C_0402" H 1403 2050 30  0001 C CNN
 F 3 "" H 1365 2200 60  0000 C CNN
 	1    1365 2200
@@
 F 0 "C39" H 1580 2300 50  0000 L CNN
 F 1 "10uF/6.3V" V 1500 1750 50  0000 L CNN
-F 2 "COMMON0603:Common_0603" H 1593 2050 30  0001 C CNN
+F 2 "Capacitors_SMD:C_0402" H 1593 2050 30  0001 C CNN
 F 3 "" H 1555 2200 60  0000 C CNN
 	1    1555 2200
@@
 F 0 "C40" H 1770 2300 50  0000 L CNN
 F 1 "0.1uF/6.3V" V 1685 1725 50  0000 L CNN
-F 2 "COMMON0603:Common_0603" H 1783 2050 30  0001 C CNN
+F 2 "Capacitors_SMD:C_0402" H 1783 2050 30  0001 C CNN
 F 3 "" H 1745 2200 60  0000 C CNN
 	1    1745 2200
@@
 F 0 "C41" H 1960 2300 50  0000 L CNN
 F 1 "10uF/6.3V" V 1880 1745 50  0000 L CNN
-F 2 "COMMON0603:Common_0603" H 1973 2050 30  0001 C CNN
+F 2 "Capacitors_SMD:C_0402" H 1973 2050 30  0001 C CNN
 F 3 "" H 1935 2200 60  0000 C CNN
 	1    1935 2200
@@
 F 0 "C42" H 2150 2300 50  0000 L CNN
 F 1 "0.1uF/6.3V" V 2270 1820 50  0000 L CNN
-F 2 "COMMON0603:Common_0603" H 2163 2050 30  0001 C CNN
+F 2 "Capacitors_SMD:C_0402" H 2163 2050 30  0001 C CNN
 F 3 "" H 2125 2200 60  0000 C CNN
 	1    2125 2200
@@
 F 0 "C43" V 1125 3310 50  0000 L CNN
 F 1 "22uF/6.3V" V 920 3040 50  0000 L CNN
-F 2 "COMMON0603:Common_0603" H 1103 3100 30  0001 C CNN
+F 2 "Capacitors_SMD:C_0402" H 1103 3100 30  0001 C CNN
 F 3 "" H 1065 3250 60  0000 C CNN
 	1    1065 3250
@@
 F 0 "C44" V 1315 3315 50  0000 L CNN
 F 1 "0.1uF/6.3V" V 1195 2770 50  0000 L CNN
-F 2 "COMMON0603:Common_0603" H 1293 3100 30  0001 C CNN
+F 2 "Capacitors_SMD:C_0402" H 1293 3100 30  0001 C CNN
 F 3 "" H 1255 3250 60  0000 C CNN
 	1    1255 3250
@@
 F 0 "C48" V 1505 3315 50  0000 L CNN
 F 1 "10uF/6.3V" V 1390 2800 50  0000 L CNN
-F 2 "COMMON0603:Common_0603" H 1483 3100 30  0001 C CNN
+F 2 "Capacitors_SMD:C_0402" H 1483 3100 30  0001 C CNN
 F 3 "" H 1445 3250 60  0000 C CNN
 	1    1445 3250
@@
 F 0 "C49" V 1695 3320 50  0000 L CNN
 F 1 "0.1uF/6.3V" V 1590 2770 50  0000 L CNN
-F 2 "COMMON0603:Common_0603" H 1673 3100 30  0001 C CNN
+F 2 "Capacitors_SMD:C_0402" H 1673 3100 30  0001 C CNN
 F 3 "" H 1635 3250 60  0000 C CNN
 	1    1635 3250
@@
 F 0 "C50" V 1885 3320 50  0000 L CNN
 F 1 "10uF/6.3V" V 1970 3025 50  0000 L CNN
-F 2 "COMMON0603:Common_0603" H 1863 3100 30  0001 C CNN
+F 2 "Capacitors_SMD:C_0402" H 1863 3100 30  0001 C CNN
 F 3 "" H 1825 3250 60  0000 C CNN
 	1    1825 3250
@@
 F 0 "R26" V 8125 6140 50  0000 C CNN
 F 1 "240R/1%" V 8170 5885 50  0000 C CNN
-F 2 "COMMON0603:Common_0603" V 8005 5955 30  0001 C CNN
+F 2 "Resistors_SMD:R_0402" V 8005 5955 30  0001 C CNN
 F 3 "" H 8075 5955 30  0000 C CNN
 	1    8075 5955
@@
 F 0 "R19" H 6835 12635 50  0000 C CNN
 F 1 "2k/1%" V 6665 12490 50  0000 C CNN
-F 2 "COMMON0603:Common_0603" V 6675 12500 30  0001 C CNN
+F 2 "Resistors_SMD:R_0402" V 6675 12500 30  0001 C CNN
 F 3 "" H 6745 12500 30  0000 C CNN
 	1    6745 12500
@@
 F 0 "R74" H 6850 13015 50  0000 C CNN
 F 1 "2k/1%" V 6665 12895 50  0000 C CNN
-F 2 "COMMON0603:Common_0603" V 6675 12895 30  0001 C CNN
+F 2 "Resistors_SMD:R_0402" V 6675 12895 30  0001 C CNN
 F 3 "" H 6745 12895 30  0000 C CNN
 	1    6745 12895
@@
 F 0 "C80" H 6980 12635 50  0000 L CNN
 F 1 "0.1uF" V 7085 12340 50  0000 L CNN
-F 2 "COMMON0603:Common_0603" H 6988 12350 30  0001 C CNN
+F 2 "Capacitors_SMD:C_0402" H 6988 12350 30  0001 C CNN
 F 3 "" H 6950 12500 60  0000 C CNN
 	1    6950 12500
@@
 F 0 "C81" H 6975 13015 50  0000 L CNN
 F 1 "0.1uF" V 7085 12735 50  0000 L CNN
-F 2 "COMMON0603:Common_0603" H 6988 12745 30  0001 C CNN
+F 2 "Capacitors_SMD:C_0402" H 6988 12745 30  0001 C CNN
 F 3 "" H 6950 12895 60  0000 C CNN
 	1    6950 12895
