File: mpu_ddr3.sch (KiCad schematic (older format))
At the start: 124 parts, among them J2 DM3AT-SF-PEJM5, P10 UART1, P17 GPIO, P18 USB_A, P19 USB_OTG, P7 LCD, P8 JTAG, P9 UART0, SW3 UBOOT, U4 a13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

Commit message: Commit before production Update4
Parts:
- C34, C43: value 22uF/6.3V -> 0.1uF/6.3V
- C42, C49: value 0.1uF/6.3V -> 22uF/6.3V
Changed lines of the file:
@@
 P 795 2200
 F 0 "C34" H 820 2300 50  0000 L CNN
-F 1 "22uF/6.3V" V 750 1750 50  0000 L CNN
+F 1 "0.1uF/6.3V" V 750 1750 50  0000 L CNN
 F 2 "Capacitors_SMD:C_0402" H 833 2050 30  0001 C CNN
 F 3 "" H 795 2200 60  0000 C CNN
@@
 P 2125 2200
 F 0 "C42" H 2150 2300 50  0000 L CNN
-F 1 "0.1uF/6.3V" V 2270 1820 50  0000 L CNN
+F 1 "22uF/6.3V" V 2270 1820 50  0000 L CNN
 F 2 "Capacitors_SMD:C_0402" H 2163 2050 30  0001 C CNN
 F 3 "" H 2125 2200 60  0000 C CNN
@@
 P 1065 3250
 F 0 "C43" V 1125 3310 50  0000 L CNN
-F 1 "22uF/6.3V" V 920 3040 50  0000 L CNN
+F 1 "0.1uF/6.3V" V 920 3040 50  0000 L CNN
 F 2 "Capacitors_SMD:C_0402" H 1103 3100 30  0001 C CNN
 F 3 "" H 1065 3250 60  0000 C CNN
@@
 P 1635 3250
 F 0 "C49" V 1695 3320 50  0000 L CNN
-F 1 "0.1uF/6.3V" V 1590 2770 50  0000 L CNN
+F 1 "22uF/6.3V" V 1590 2770 50  0000 L CNN
 F 2 "Capacitors_SMD:C_0402" H 1673 3100 30  0001 C CNN
 F 3 "" H 1635 3250 60  0000 C CNN

Commit message: Fix : fix line width for impedance matching
Parts:
- P18: footprint Connect:USB_A_Vertical -> MyConnector:USB_A_Vertical
- P19: footprint Connect:USB_Micro-B -> MyConnector:USB_Micro-B
Changed lines of the file:
@@
 F 0 "P18" V 4445 13620 50  0000 C CNN
 F 1 "USB_A" H 4685 13815 50  0000 C CNN
-F 2 "Connect:USB_A_Vertical" V 4685 13515 60  0001 C CNN
+F 2 "MyConnector:USB_A_Vertical" V 4685 13515 60  0001 C CNN
 F 3 "" V 4685 13515 60  0000 C CNN
 	1    4735 13615
@@
 F 0 "P19" V 4489 15085 50  0000 C CNN
 F 1 "USB_OTG" H 4789 15285 50  0000 C CNN
-F 2 "Connect:USB_Micro-B" V 4739 14985 60  0001 C CNN
+F 2 "MyConnector:USB_Micro-B" V 4739 14985 60  0001 C CNN
 F 3 "" V 4739 14985 60  0000 C CNN
 	1    4789 15085
