File: gc3.sch (KiCad schematic (older format))
At the start: 67 parts, among them J1 JACK_2P, P1 TESTPOINT, P11 CONN_01X01, P12 CONN_01X01, P13 CONN_01X01, P14 CONN_01X01, P15 TESTPOINT, P16 TESTPOINT, P2 TESTPOINT, P3 TESTPOINT, P4 TESTPOINT, P5 TESTPOINT, P6 TESTPOINT, SW1 PWR_ON, SW2 RESET, U1 TPS62290, U2 axp209, U3 TPS62290

Commit message: clean sch and add resistor array
Parts:
- removed C1: 120uF/16V, SMD_Packages:SMD-0603_c, symbol CP2
- removed C10, C3: 4.7uF, symbol C-RESCUE-gc3
- removed C11, C14: 22pF, symbol C-RESCUE-gc3
- removed C12, C13, C15, C16, C17, C18, C19, C22, C23, C4, C5, C6, C8: 10uF/6.3V, SMD_Packages:SMD-0603_c, symbol C-RESCUE-gc3
- removed C2, C9: 1uF, SMD_Packages:SMD-0603_c, symbol C-RESCUE-gc3
- removed C20: NA or 10uF/6.3V, SMD_Packages:SMD-0603_c, symbol C-RESCUE-gc3
- removed C21, C26: 10uF, symbol C-RESCUE-gc3
- removed C24, C25, C7: 1nF, SMD_Packages:SMD-0603_c, symbol C-RESCUE-gc3
- removed C27, C37: 100uF/25V, symbol CP2
- removed D1: DIODE, symbol DIODE
- removed JP1: JUMPER, symbol R-RESCUE-gc3
- removed L1, L4: 2.2uH, symbol INDUCTOR
- removed L2, L3: 2.2uH/1.5A, symbol INDUCTOR
- removed R1: 510R, symbol R-RESCUE-gc3
- removed R10, R3: 2.2k, symbol R-RESCUE-gc3
- removed R11: 360k, symbol R-RESCUE-gc3
- removed R12: 100K, symbol R-RESCUE-gc3
- removed R13: 22K, symbol R-RESCUE-gc3
- removed R2: 540k, symbol R-RESCUE-gc3
- removed R4: 1k, symbol R-RESCUE-gc3
- removed R5: 240R/1%, symbol R-RESCUE-gc3
- removed R6, R7: 1R, symbol R-RESCUE-gc3
- removed R8: 47k, symbol R-RESCUE-gc3
- removed R9: 200k/1%, symbol R-RESCUE-gc3
- added C1: 120uF/16V, Capacitors_ThroughHole:C_Radial_D5_L11_P2, symbol CP
- added C10, C3: 4.7uF, Capacitors_SMD:C_0603, symbol C
- added C11, C14: 22pF, Capacitors_SMD:C_0603, symbol C
- added C12, C13, C15, C16, C17, C18, C19, C20, C22, C23, C4, C5, C6, C8: 10uF/6.3V, Capacitors_SMD:C_0603, symbol C
- added C2, C9: 1uF, Capacitors_SMD:C_0603, symbol C
- added C21, C26: 10uF, Capacitors_SMD:C_0603, symbol C
- added C24, C25, C7: 1nF, Capacitors_SMD:C_0603, symbol C
- added C27, C37: 100uF, Capacitors_ThroughHole:C_Radial_D5_L11_P2, symbol CP
- added D1: DIODE, Diodes_SMD:SOD-123, symbol D
- added JP1: JUMPER, Resistors_SMD:R_0603, symbol R
- added L1, L4: 2.2uH, Inductors_NEOSID:Neosid_Inductor_SMS-ME3015, symbol INDUCTOR_SMALL
- added L2, L3: 2.2uH, ELL4LG2R2NA:ELL4LG2R2NA, symbol INDUCTOR_SMALL
- added R1: 510R, Resistors_SMD:R_0603, symbol R
- added R10, R3: 2.2k, Resistors_SMD:R_0603, symbol R
- added R11: 360k, Resistors_SMD:R_0603, symbol R
- added R12: 100k, Resistors_SMD:R_0603, symbol R
- added R13: 22k, Resistors_SMD:R_0603, symbol R
- added R2: 540k, Resistors_SMD:R_0603, symbol R
- added R4: 1k, Resistors_SMD:R_0603, symbol R
- added R5: 240R/1%, Resistors_SMD:R_0603, symbol R
- added R6, R7: 1R, Resistors_SMD:R_0603, symbol R
- added R8: 47k, Resistors_SMD:R_0603, symbol R
- added R9: 200k/1%, Resistors_SMD:R_0603, symbol R
- D2: value PWR -> LED; footprint (none) -> LEDs:LED-0805
- J1: value JACK_2P -> JACK; footprint (none) -> Connect:BARREL_JACK
- P1: footprint (none) -> Measurement_Points:Measurement_Point_Round-SMD-Pad_Small
- P11, P12, P13, P14: value CONN_01X01 -> GND; footprint (none) -> SMD_Packages:1Pin
- P15, P2, P3, P4, P5, P6: footprint Pin_Headers:Pin_Header_Straight_1x01 -> Measurement_Points:Measurement_Point_Round-SMD-Pad_Small
- P16: value TESTPOINT -> TEESTPOINT; footprint (none) -> Measurement_Points:Measurement_Point_Round-SMD-Pad_Small
- R15: footprint (none) -> Resistors_SMD:R_0603
- SW1, SW2: footprint (none) -> Buttons_Switches_SMD:SW_SPST_FSMSM
- U1, U3: footprint (none) -> TPS62290:TPS62290
- U2: footprint (none) -> AXP209:TQFP-48-1EP_6x6mm_Pitch0.4mm
Connections:
- wire segments 183 -> 186
Other:
- note removed: "3.3v"
- note removed: "defalt open/not use"

Commit message: commit before cleanup all footprint
Parts:
- D2: value LED -> POWER
- L2, L3: footprint ELL4LG2R2NA:ELL4LG2R2NA -> Inductors_NEOSID:Neosid_Inductor_SMS-ME3015
Changed lines of the file:
@@
 LIBS:valves
 LIBS:a13
-LIBS:mp1482ds
 LIBS:3.0VA
 LIBS:1.2V_CPU
 LIBS:1.2V_INT
 LIBS:+1.5V
-LIBS:pcf8563t5
 LIBS:usd
 LIBS:axp209
@@
 LIBS:crystall
 LIBS:resistorarray
+LIBS:blueninja
 LIBS:gc3-cache
 EELAYER 25 0
@@
 U 1 1 56AF4055
 P 12385 1795
-F 0 "C1" H 12410 1895 50  0000 L CNN
+F 0 "C1" H 12230 1935 50  0000 L CNN
 F 1 "120uF/16V" V 12455 1315 50  0000 L CNN
 F 2 "Capacitors_ThroughHole:C_Radial_D5_L11_P2" H 12423 1645 30  0001 C CNN
@@
 U 1 1 56AF4711
 P 12885 1755
-F 0 "R15" V 12965 1755 50  0000 C CNN
+F 0 "R15" H 12755 1845 50  0000 C CNN
 F 1 "90R" V 12885 1755 50  0000 C CNN
 F 2 "Resistors_SMD:R_0603" V 12815 1755 30  0001 C CNN
@@
 U 1 1 56AF4B4B
 P 12885 2180
-F 0 "D2" H 12885 2280 50  0000 C CNN
-F 1 "LED" H 12885 2080 50  0000 C CNN
+F 0 "D2" V 12965 2310 50  0000 C CNN
+F 1 "POWER" V 12895 1965 50  0000 C CNN
 F 2 "LEDs:LED-0805" H 12885 2180 60  0001 C CNN
 F 3 "" H 12885 2180 60  0000 C CNN
@@
 L GND #PWR021
 U 1 1 5616F10F
-P 2970 2325
-F 0 "#PWR021" H 2970 2075 50  0001 C CNN
-F 1 "GND" V 2970 2130 50  0000 C CNN
-F 2 "" H 2970 2325 60  0000 C CNN
-F 3 "" H 2970 2325 60  0000 C CNN
-	1    2970 2325
+P 2920 2325
+F 0 "#PWR021" H 2920 2075 50  0001 C CNN
+F 1 "GND" V 2920 2130 50  0000 C CNN
+F 2 "" H 2920 2325 60  0000 C CNN
+F 3 "" H 2920 2325 60  0000 C CNN
+	1    2920 2325
 	0    1    1    0
 $EndComp
@@
 F 0 "L2" H 6910 3265 50  0000 C CNN
 F 1 "2.2uH" H 7485 3265 50  0000 C CNN
-F 2 "ELL4LG2R2NA:ELL4LG2R2NA" H 7170 3225 60  0001 C CNN
+F 2 "Inductors_NEOSID:Neosid_Inductor_SMS-ME3015" H 7170 3225 60  0001 C CNN
 F 3 "" H 7170 3225 60  0000 C CNN
 	1    7170 3225
@@
 F 0 "L3" H 6920 3975 50  0000 C CNN
 F 1 "2.2uH" H 7510 3975 50  0000 C CNN
-F 2 "ELL4LG2R2NA:ELL4LG2R2NA" H 7185 3925 60  0001 C CNN
+F 2 "Inductors_NEOSID:Neosid_Inductor_SMS-ME3015" H 7185 3925 60  0001 C CNN
 F 3 "" H 7185 3925 60  0000 C CNN
 	1    7185 3925
@@
 L GND #PWR032
 U 1 1 5622813C
-P 2970 3125
-F 0 "#PWR032" H 2970 2875 50  0001 C CNN
-F 1 "GND" H 2970 2975 50  0000 C CNN
-F 2 "" H 2970 3125 60  0000 C CNN
-F 3 "" H 2970 3125 60  0000 C CNN
-	1    2970 3125
+P 2920 3125
+F 0 "#PWR032" H 2920 2875 50  0001 C CNN
+F 1 "GND" H 2920 2975 50  0000 C CNN
+F 2 "" H 2920 3125 60  0000 C CNN
+F 3 "" H 2920 3125 60  0000 C CNN
+	1    2920 3125
 	0    1    1    0
 $EndComp
@@
 NoConn ~ 4380 3825
 Wire Wire Line
-	3055 3125 2970 3125
-Wire Wire Line
 	4380 2325 3705 2325
 Wire Wire Line
@@
 	3705 3125 4380 3125
 Connection ~ 4015 3125
-Wire Wire Line
-	3405 2325 2970 2325
 $Comp
 L C C8
@@
 Connection ~ 13580 5605
 Connection ~ 13600 3585
+Wire Wire Line
+	3055 3125 2920 3125
+Wire Wire Line
+	3405 2325 2920 2325
 $EndSCHEMATC

Commit message: GC3-Update3
Parts:
- R11: value 360k -> 210k
- R2: value 540k -> 315k
Changed lines of the file:
@@
 P 12685 5815
 F 0 "R2" H 12575 5705 50  0000 C CNN
-F 1 "540k" V 12685 5815 50  0000 C CNN
+F 1 "315k" V 12685 5815 50  0000 C CNN
 F 2 "Resistors_SMD:R_0603" V 12615 5815 30  0001 C CNN
 F 3 "" H 12685 5815 30  0000 C CNN
@@
 P 12685 6180
 F 0 "R11" H 12565 6095 50  0000 C CNN
-F 1 "360k" V 12685 6180 50  0000 C CNN
+F 1 "210k" V 12685 6180 50  0000 C CNN
 F 2 "Resistors_SMD:R_0603" V 12615 6180 30  0001 C CNN
 F 3 "" H 12685 6180 30  0000 C CNN
@@
 	10990 5855 10990 6430
 Wire Wire Line
-	11165 5955 10990 5955
-Connection ~ 10990 5955
-Wire Wire Line
 	12685 5665 12685 5605
 Connection ~ 12685 5605
@@
 Wire Wire Line
 	11010 3835 11010 4410
-Wire Wire Line
-	11185 3935 11010 3935
-Connection ~ 11010 3935
 Wire Wire Line
 	12705 3645 12705 3585
@@
 	7450 4525 7315 4525
 Wire Wire Line
-	7015 4525 6280 4525
+	6280 4525 7015 4525
 Wire Wire Line
 	6280 4225 6900 4225
@@
 $EndComp
 Wire Wire Line
-	4380 3225 4015 3225
-Wire Wire Line
-	4015 3225 4015 1915
+	4015 3225 4380 3225
+Wire Wire Line
+	4015 1915 4015 3225
 $Comp
 L R R6
@@
 $EndComp
 Wire Wire Line
-	4380 2825 3355 2825
+	3355 2825 4380 2825
 $Comp
 L GND #PWR033
@@
 $EndComp
 Wire Wire Line
-	4380 3525 3705 3525
+	3705 3525 4380 3525
 Wire Wire Line
 	3405 3525 3355 3525
@@
 $EndComp
 Wire Wire Line
-	4380 5725 3355 5725
+	3355 5725 4380 5725
 $Comp
 L R R4
@@
 $EndComp
 Wire Wire Line
-	3055 5725 2920 5725
+	2920 5725 3055 5725
 Wire Wire Line
 	3055 5470 2995 5470
@@
 $EndComp
 Wire Wire Line
-	4380 6325 3655 6325
+	3655 6325 4380 6325
 $Comp
 L R R3
@@
 $EndComp
 Wire Wire Line
-	4380 6425 3655 6425
-Wire Wire Line
-	3355 6325 2920 6325
+	3655 6425 4380 6425
+Wire Wire Line
+	2920 6325 3355 6325
 Wire Wire Line
 	3355 6425 3000 6425
@@
 Wire Wire Line
 	3405 2325 2920 2325
+Wire Wire Line
+	11185 3935 11084 3935
+Wire Wire Line
+	11165 5955 11041 5955
+Text Label 11148 3935 2    60   ~ 0
+IPSOUT
+Text Label 11114 5955 2    60   ~ 0
+IPSOUT
 $EndSCHEMATC

Commit message: Fix : bug fix
Parts:
- C1: value 120uF/16V -> 100uF
- P11, P12, P13, P14: footprint SMD_Packages:1Pin -> Connect:1pin
Changed lines of the file:
@@
 P 12385 1795
 F 0 "C1" H 12230 1935 50  0000 L CNN
-F 1 "120uF/16V" V 12455 1315 50  0000 L CNN
+F 1 "100uF" V 12452 1498 50  0000 L CNN
 F 2 "Capacitors_ThroughHole:C_Radial_D5_L11_P2" H 12423 1645 30  0001 C CNN
 F 3 "" H 12385 1795 60  0000 C CNN
@@
 F 0 "P11" H 3720 8560 50  0000 C CNN
 F 1 "GND" H 3860 8435 50  0000 C CNN
-F 2 "SMD_Packages:1Pin" H 3720 8460 60  0001 C CNN
+F 2 "Connect:1pin" H 3720 8460 60  0001 C CNN
 F 3 "" H 3720 8460 60  0000 C CNN
 	1    3720 8460
@@
 F 0 "P12" H 3715 8795 50  0000 C CNN
 F 1 "GND" H 3860 8670 50  0000 C CNN
-F 2 "SMD_Packages:1Pin" H 3715 8695 60  0001 C CNN
+F 2 "Connect:1pin" H 3715 8695 60  0001 C CNN
 F 3 "" H 3715 8695 60  0000 C CNN
 	1    3715 8695
@@
 F 0 "P13" H 3720 9040 50  0000 C CNN
 F 1 "GND" H 3855 8925 50  0000 C CNN
-F 2 "SMD_Packages:1Pin" H 3720 8940 60  0001 C CNN
+F 2 "Connect:1pin" H 3720 8940 60  0001 C CNN
 F 3 "" H 3720 8940 60  0000 C CNN
 	1    3720 8940
@@
 F 0 "P14" H 3720 9285 50  0000 C CNN
 F 1 "GND" H 3795 9165 50  0000 L CNN
-F 2 "SMD_Packages:1Pin" H 3720 9185 60  0001 C CNN
+F 2 "Connect:1pin" H 3720 9185 60  0001 C CNN
 F 3 "" H 3720 9185 60  0000 C CNN
 	1    3720 9185

Commit message: Temp : Temp commit for before Update4
Parts:
- C10, C11, C12, C13, C14, C15, C16, C17, C18, C19, C2, C20, C21, C22, C23, C24, C25, C26, C3, C4, C5, C6, C7, C8, C9: footprint Capacitors_SMD:C_0603 -> COMMON0603:Common_0603
- R1, R10, R11, R12, R13, R15, R2, R3, R4, R5, R6, R7, R8, R9: footprint Resistors_SMD:R_0603 -> COMMON0603:Common_0603
Changed lines of the file:
@@
 F 0 "R15" H 12755 1845 50  0000 C CNN
 F 1 "90R" V 12885 1755 50  0000 C CNN
-F 2 "Resistors_SMD:R_0603" V 12815 1755 30  0001 C CNN
+F 2 "COMMON0603:Common_0603" V 12815 1755 30  0001 C CNN
 F 3 "" H 12885 1755 30  0000 C CNN
 	1    12885 1755
@@
 F 0 "C3" H 10790 6080 50  0000 L CNN
 F 1 "4.7uF" V 10700 5710 50  0000 L CNN
-F 2 "Capacitors_SMD:C_0603" H 10803 5830 30  0001 C CNN
+F 2 "COMMON0603:Common_0603" H 10803 5830 30  0001 C CNN
 F 3 "" H 10765 5980 60  0000 C CNN
 	1    10765 5980
@@
 F 0 "R2" H 12575 5705 50  0000 C CNN
 F 1 "315k" V 12685 5815 50  0000 C CNN
-F 2 "Resistors_SMD:R_0603" V 12615 5815 30  0001 C CNN
+F 2 "COMMON0603:Common_0603" V 12615 5815 30  0001 C CNN
 F 3 "" H 12685 5815 30  0000 C CNN
 	1    12685 5815
@@
 F 0 "R11" H 12565 6095 50  0000 C CNN
 F 1 "210k" V 12685 6180 50  0000 C CNN
-F 2 "Resistors_SMD:R_0603" V 12615 6180 30  0001 C CNN
+F 2 "COMMON0603:Common_0603" V 12615 6180 30  0001 C CNN
 F 3 "" H 12685 6180 30  0000 C CNN
 	1    12685 6180
@@
 F 0 "C11" H 12965 5915 50  0000 L CNN
 F 1 "22pF" V 13005 5565 50  0000 L CNN
-F 2 "Capacitors_SMD:C_0603" H 12978 5665 30  0001 C CNN
+F 2 "COMMON0603:Common_0603" H 12978 5665 30  0001 C CNN
 F 3 "" H 12940 5815 60  0000 C CNN
 	1    12940 5815
@@
 F 0 "C21" H 13330 5905 50  0000 L CNN
 F 1 "10uF" V 13275 5575 50  0000 L CNN
-F 2 "Capacitors_SMD:C_0603" H 13353 5665 30  0001 C CNN
+F 2 "COMMON0603:Common_0603" H 13353 5665 30  0001 C CNN
 F 3 "" H 13315 5815 60  0000 C CNN
 	1    13315 5815
@@
 F 0 "C10" H 10810 4060 50  0000 L CNN
 F 1 "4.7uF" V 10720 3690 50  0000 L CNN
-F 2 "Capacitors_SMD:C_0603" H 10823 3810 30  0001 C CNN
+F 2 "COMMON0603:Common_0603" H 10823 3810 30  0001 C CNN
 F 3 "" H 10785 3960 60  0000 C CNN
 	1    10785 3960
@@
 F 0 "R12" H 12595 3685 50  0000 C CNN
 F 1 "100k" V 12705 3795 50  0000 C CNN
-F 2 "Resistors_SMD:R_0603" V 12635 3795 30  0001 C CNN
+F 2 "COMMON0603:Common_0603" V 12635 3795 30  0001 C CNN
 F 3 "" H 12705 3795 30  0000 C CNN
 	1    12705 3795
@@
 F 0 "R13" H 12585 4075 50  0000 C CNN
 F 1 "22k" V 12705 4160 50  0000 C CNN
-F 2 "Resistors_SMD:R_0603" V 12635 4160 30  0001 C CNN
+F 2 "COMMON0603:Common_0603" V 12635 4160 30  0001 C CNN
 F 3 "" H 12705 4160 30  0000 C CNN
 	1    12705 4160
@@
 F 0 "C14" H 12985 3895 50  0000 L CNN
 F 1 "22pF" V 13025 3545 50  0000 L CNN
-F 2 "Capacitors_SMD:C_0603" H 12998 3645 30  0001 C CNN
+F 2 "COMMON0603:Common_0603" H 12998 3645 30  0001 C CNN
 F 3 "" H 12960 3795 60  0000 C CNN
 	1    12960 3795
@@
 F 0 "C26" H 13350 3885 50  0000 L CNN
 F 1 "10uF" V 13295 3555 50  0000 L CNN
-F 2 "Capacitors_SMD:C_0603" H 13373 3645 30  0001 C CNN
+F 2 "COMMON0603:Common_0603" H 13373 3645 30  0001 C CNN
 F 3 "" H 13335 3795 60  0000 C CNN
 	1    13335 3795
@@
 F 0 "R5" V 3515 2490 50  0000 C CNN
 F 1 "240R/1%" V 3520 2040 50  0000 C CNN
-F 2 "Resistors_SMD:R_0603" V 3485 2325 30  0001 C CNN
+F 2 "COMMON0603:Common_0603" V 3485 2325 30  0001 C CNN
 F 3 "" H 3555 2325 30  0000 C CNN
 	1    3555 2325
@@
 F 0 "C15" V 7120 2530 50  0000 L CNN
 F 1 "10uF/6.3V" V 7125 2810 50  0000 L CNN
-F 2 "Capacitors_SMD:C_0603" H 7203 2575 30  0001 C CNN
+F 2 "COMMON0603:Common_0603" H 7203 2575 30  0001 C CNN
 F 3 "" H 7165 2725 60  0000 C CNN
 	1    7165 2725
@@
 F 0 "C12" V 7120 3125 50  0000 L CNN
 F 1 "10uF/6.3V" V 7120 3410 50  0000 L CNN
-F 2 "Capacitors_SMD:C_0603" H 7203 3175 30  0001 C CNN
+F 2 "COMMON0603:Common_0603" H 7203 3175 30  0001 C CNN
 F 3 "" H 7165 3325 60  0000 C CNN
 	1    7165 3325
@@
 F 0 "C13" V 7125 3930 50  0000 L CNN
 F 1 "10uF/6.3V" V 7300 3915 50  0000 L CNN
-F 2 "Capacitors_SMD:C_0603" H 7203 3975 30  0001 C CNN
+F 2 "COMMON0603:Common_0603" H 7203 3975 30  0001 C CNN
 F 3 "" H 7165 4125 60  0000 C CNN
 	1    7165 4125
@@
 F 0 "C18" V 7120 4330 50  0000 L CNN
 F 1 "10uF/6.3V" V 7120 4590 50  0000 L CNN
-F 2 "Capacitors_SMD:C_0603" H 7203 4375 30  0001 C CNN
+F 2 "COMMON0603:Common_0603" H 7203 4375 30  0001 C CNN
 F 3 "" H 7165 4525 60  0000 C CNN
 	1    7165 4525
@@
 F 0 "C19" V 7120 4540 50  0000 L CNN
 F 1 "10uF/6.3V" V 7120 4790 50  0000 L CNN
-F 2 "Capacitors_SMD:C_0603" H 7203 4575 30  0001 C CNN
+F 2 "COMMON0603:Common_0603" H 7203 4575 30  0001 C CNN
 F 3 "" H 7165 4725 60  0000 C CNN
 	1    7165 4725
@@
 F 0 "C16" V 7125 4740 50  0000 L CNN
 F 1 "10uF/6.3V" V 7120 4995 50  0000 L CNN
-F 2 "Capacitors_SMD:C_0603" H 7203 4775 30  0001 C CNN
+F 2 "COMMON0603:Common_0603" H 7203 4775 30  0001 C CNN
 F 3 "" H 7165 4925 60  0000 C CNN
 	1    7165 4925
@@
 F 0 "C17" V 7120 4935 50  0000 L CNN
 F 1 "10uF/6.3V" V 7115 5190 50  0000 L CNN
-F 2 "Capacitors_SMD:C_0603" H 7203 4975 30  0001 C CNN
+F 2 "COMMON0603:Common_0603" H 7203 4975 30  0001 C CNN
 F 3 "" H 7165 5125 60  0000 C CNN
 	1    7165 5125
@@
 F 0 "C20" V 7125 5135 50  0000 L CNN
 F 1 "10uF/6.3V" V 7125 5390 50  0000 L CNN
-F 2 "Capacitors_SMD:C_0603" H 7203 5175 30  0001 C CNN
+F 2 "COMMON0603:Common_0603" H 7203 5175 30  0001 C CNN
 F 3 "" H 7165 5325 60  0000 C CNN
 	1    7165 5325
@@
 F 0 "C23" H 8000 3540 50  0000 L CNN
 F 1 "10uF/6.3V" H 7560 3325 50  0000 L CNN
-F 2 "Capacitors_SMD:C_0603" H 8013 3290 30  0001 C CNN
+F 2 "COMMON0603:Common_0603" H 8013 3290 30  0001 C CNN
 F 3 "" H 7975 3440 60  0000 C CNN
 	1    7975 3440
@@
 F 0 "C24" H 8205 3540 50  0000 L CNN
 F 1 "1nF" H 8205 3340 50  0000 L CNN
-F 2 "Capacitors_SMD:C_0603" H 8218 3290 30  0001 C CNN
+F 2 "COMMON0603:Common_0603" H 8218 3290 30  0001 C CNN
 F 3 "" H 8180 3440 60  0000 C CNN
 	1    8180 3440
@@
 F 0 "C22" H 7995 4240 50  0000 L CNN
 F 1 "10uF/6.3V" H 7550 4020 50  0000 L CNN
-F 2 "Capacitors_SMD:C_0603" H 8008 3990 30  0001 C CNN
+F 2 "COMMON0603:Common_0603" H 8008 3990 30  0001 C CNN
 F 3 "" H 7970 4140 60  0000 C CNN
 	1    7970 4140
@@
 F 0 "C25" H 8215 4240 50  0000 L CNN
 F 1 "1nF" H 8215 4040 50  0000 L CNN
-F 2 "Capacitors_SMD:C_0603" H 8228 3990 30  0001 C CNN
+F 2 "COMMON0603:Common_0603" H 8228 3990 30  0001 C CNN
 F 3 "" H 8190 4140 60  0000 C CNN
 	1    8190 4140
@@
 F 0 "R6" V 3525 3280 50  0000 C CNN
 F 1 "1R" V 3555 3125 50  0000 C CNN
-F 2 "Resistors_SMD:R_0603" V 3485 3125 30  0001 C CNN
+F 2 "COMMON0603:Common_0603" V 3485 3125 30  0001 C CNN
 F 3 "" H 3555 3125 30  0000 C CNN
 	1    3555 3125
@@
 F 0 "C6" V 3160 3200 50  0000 L CNN
 F 1 "10uF/6.3V" V 3340 2965 50  0000 L CNN
-F 2 "Capacitors_SMD:C_0603" H 3243 2975 30  0001 C CNN
+F 2 "COMMON0603:Common_0603" H 3243 2975 30  0001 C CNN
 F 3 "" H 3205 3125 60  0000 C CNN
 	1    3205 3125
@@
 F 0 "C8" V 3160 2900 50  0000 L CNN
 F 1 "10uF/6.3V" V 3265 2875 50  0000 L CNN
-F 2 "Capacitors_SMD:C_0603" H 3243 2675 30  0001 C CNN
+F 2 "COMMON0603:Common_0603" H 3243 2675 30  0001 C CNN
 F 3 "" H 3205 2825 60  0000 C CNN
 	1    3205 2825
@@
 F 0 "C4" V 3160 3590 50  0000 L CNN
 F 1 "10uF/6.3V" V 3335 3335 50  0000 L CNN
-F 2 "Capacitors_SMD:C_0603" H 3243 3375 30  0001 C CNN
+F 2 "COMMON0603:Common_0603" H 3243 3375 30  0001 C CNN
 F 3 "" H 3205 3525 60  0000 C CNN
 	1    3205 3525
@@
 F 0 "R7" V 3505 3680 50  0000 C CNN
 F 1 "1R" V 3555 3525 50  0000 C CNN
-F 2 "Resistors_SMD:R_0603" V 3485 3525 30  0001 C CNN
+F 2 "COMMON0603:Common_0603" V 3485 3525 30  0001 C CNN
 F 3 "" H 3555 3525 30  0000 C CNN
 	1    3555 3525
@@
 F 0 "C2" V 3160 4700 50  0000 L CNN
 F 1 "1uF" V 3250 4435 50  0000 L CNN
-F 2 "Capacitors_SMD:C_0603" H 3243 4475 30  0001 C CNN
+F 2 "COMMON0603:Common_0603" H 3243 4475 30  0001 C CNN
 F 3 "" H 3205 4625 60  0000 C CNN
 	1    3205 4625
@@
 F 0 "R9" V 3520 4900 50  0000 C CNN
 F 1 "200k/1%" V 3640 4730 50  0000 C CNN
-F 2 "Resistors_SMD:R_0603" V 3485 4725 30  0001 C CNN
+F 2 "COMMON0603:Common_0603" V 3485 4725 30  0001 C CNN
 F 3 "" H 3555 4725 30  0000 C CNN
 	1    3555 4725
@@
 F 0 "C9" V 3165 4990 50  0000 L CNN
 F 1 "1uF" V 3260 4740 50  0000 L CNN
-F 2 "Capacitors_SMD:C_0603" H 3243 4775 30  0001 C CNN
+F 2 "COMMON0603:Common_0603" H 3243 4775 30  0001 C CNN
 F 3 "" H 3205 4925 60  0000 C CNN
 	1    3205 4925
@@
 F 0 "C5" V 3580 5130 50  0000 L CNN
 F 1 "10uF/6.3V" V 3680 4615 50  0000 L CNN
-F 2 "Capacitors_SMD:C_0603" H 3663 4925 30  0001 C CNN
+F 2 "COMMON0603:Common_0603" H 3663 4925 30  0001 C CNN
 F 3 "" H 3625 5075 60  0000 C CNN
 	1    3625 5075
@@
 F 0 "C7" V 3160 5805 50  0000 L CNN
 F 1 "1nF" V 3255 5795 50  0000 L CNN
-F 2 "Capacitors_SMD:C_0603" H 3243 5575 30  0001 C CNN
+F 2 "COMMON0603:Common_0603" H 3243 5575 30  0001 C CNN
 F 3 "" H 3205 5725 60  0000 C CNN
 	1    3205 5725
@@
 F 0 "R4" V 3820 5635 50  0000 C CNN
 F 1 "1k" V 3865 5470 50  0000 C CNN
-F 2 "Resistors_SMD:R_0603" V 3795 5470 30  0001 C CNN
+F 2 "COMMON0603:Common_0603" V 3795 5470 30  0001 C CNN
 F 3 "" H 3865 5470 30  0000 C CNN
 	1    3865 5470
@@
 F 0 "R8" V 3685 7080 50  0000 C CNN
 F 1 "47k" V 3605 7080 50  0000 C CNN
-F 2 "Resistors_SMD:R_0603" V 3535 7080 30  0001 C CNN
+F 2 "COMMON0603:Common_0603" V 3535 7080 30  0001 C CNN
 F 3 "" H 3605 7080 30  0000 C CNN
 	1    3605 7080
@@
 F 0 "R10" V 3470 6515 50  0000 C CNN
 F 1 "2.2k" V 3505 6325 50  0000 C CNN
-F 2 "Resistors_SMD:R_0603" V 3435 6325 30  0001 C CNN
+F 2 "COMMON0603:Common_0603" V 3435 6325 30  0001 C CNN
 F 3 "" H 3505 6325 30  0000 C CNN
 	1    3505 6325
@@
 F 0 "R3" V 3475 6590 50  0000 C CNN
 F 1 "2.2k" V 3510 6425 50  0000 C CNN
-F 2 "Resistors_SMD:R_0603" V 3435 6425 30  0001 C CNN
+F 2 "COMMON0603:Common_0603" V 3435 6425 30  0001 C CNN
 F 3 "" H 3505 6425 30  0000 C CNN
 	1    3505 6425
@@
 F 0 "R1" V 3835 5860 50  0000 C CNN
 F 1 "510R" V 3890 6025 50  0000 C CNN
-F 2 "Resistors_SMD:R_0603" V 3820 6025 30  0001 C CNN
+F 2 "COMMON0603:Common_0603" V 3820 6025 30  0001 C CNN
 F 3 "" H 3890 6025 30  0000 C CNN
 	1    3890 6025

Commit message: Fix : fix line width for impedance matching
Parts:
- J1: footprint Connect:BARREL_JACK -> MyConnector:BARREL_JACK
Changed lines of the file:
@@
 F 0 "J1" H 11210 1470 50  0000 C CNN
 F 1 "JACK" H 11410 1920 50  0000 C CNN
-F 2 "Connect:BARREL_JACK" H 11560 1670 60  0001 C CNN
+F 2 "MyConnector:BARREL_JACK" H 11560 1670 60  0001 C CNN
 F 3 "" H 11560 1670 60  0000 C CNN
 	1    11560 1670
